File: oresat-camera-hardware/AR0130_DEV_BOARD/AR0130_DEV_BOARD.sch (EAGLE design)
At the start: 61 parts, among them J2 4-1734592-0, U0 AR0130CSSM00SPCA0−DRBR1-847AC, U10 SN74AVCB164245VR, U11 KC2520B27.0000C10E00, U12 TPS71818-33DRVT, U13 SN74AVCH8T245RHLR, U14 TPS71928-28DRVT, U15 TPS71928-28DRVT, U6 MCP9808T-E/MCDFN8_2X3MC-M, U7 MCP9808T-E/MCDFN8_2X3MC-M, U9 TCA9509DGKRDGK8-M

Commit message: schematic and board revisions after design review with AG
Connections:
- removed net N$1: U7.ALERT
- removed net N$29: U0.37-NC
- removed net N$30: U0.36-NC
- removed net N$31: U0.35-NC
- removed net N$6: U6.ALERT
Other:
- moved on the sheet: C1, C13, C14, C15, C19, C2, C20, C21, C22, C23, C24, C25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

Commit message: more updates to schematic
Parts:
- removed TP7: TPTP06R, testpad:TPTP06R
- removed U0: AR0130CSSM00SPCA0−DRBR1-847AC, Oliver_Custom:AR0130CSSM00SPCA0−DRBR1-847AC
- added U$2: AR0130CSSM00SPCA0−DRBR1-847AC, Oliver_Custom:AR0130CSSM00SPCA0−DRBR1-847AC
Connections:
- removed net D0_I: U0.28-DOUT0, U10.1B1
- removed net D10_I: U0.18-DOUT10, U10.2B3
- removed net D11_I: U0.17-DOUT11, U10.2B4
- removed net D1_I: U0.27-DOUT1, U10.1B2
- removed net D2_I: U0.26-DOUT2, U10.1B3
- removed net D3_I: U0.25-DOUT3, U10.1B4
- removed net D4_I: U0.24-DOUT4, U10.1B5
- removed net D5_I: U0.23-DOUT5, U10.1B6
- removed net D6_I: U0.22-DOUT6, U10.1B7
- removed net D7_I: U0.21-DOUT7, U10.1B8
- removed net D8_I: U0.20-DOUT8, U10.2B1
- removed net D9_I: U0.19-DOUT9, U10.2B2
- removed net HSYNC_I: U0.16-LINEVALID, U10.2B5
- removed net N$56: R1.2, U0.11-EXTCLK
- removed net N$71: U10.2B8
- removed net N$95: U10.2A8
- removed net PIXCLK_I: U0.12-PIXCLK, U10.2B7
- removed net VSYNC_I: U0.15-FRAME_VALID, U10.2B6
- new net 1.8V: C1.1, C19.1, U$2.VDD
- new net 2.8V: C2.1, C20.1, U$2.VDD_IO, U10.VCCB, U10.VCCB_2
- new net DI_0: U$2.DOUT0, U10.1B1
- new net DI_1: U$2.DOUT1, U10.1B2
- new net DI_10: U$2.DOUT10, U10.2B3
- new net DI_11: U$2.DOUT11, U10.2B4
- new net DI_2: U$2.DOUT2, U10.1B3
- new net DI_3: U$2.DOUT3, U10.1B4
- new net DI_4: U$2.DOUT4, U$2.DOUT5, U10.1B5
- new net DI_5: U10.1B6
- new net DI_6: U$2.DOUT6, U10.1B7
- new net DI_7: U$2.DOUT7, U10.1B8
- new net DI_8: U$2.DOUT8, U10.2B1
- new net DI_9: U$2.DOUT9, U10.2B2
- new net HSYNC: U$2.LINEVALID, U10.2B5
- new net N$1: R1.2, U$2.EXTCLK
- new net N$10: U$2.OE_BAR
- new net N$11: U$2.RESET_BAR
- new net N$5: U$2.SADDR
- new net N$6: U$2.SCLK
- new net N$8: U$2.SDATA
- new net N$9: U$2.TRIGGER
- new net PIXCLK: U$2.PIXCLK, U10.2B7
- new net VCC: C21.1, C3.1, U$2.VAA
- new net VCC_1: C22.1, C4.1, U$2.VDD_PLL
- new net VCC_2: C23.1, C5.1, U$2.VAA_PIX
- new net VSYNC: U$2.FRAME_VALID, U10.2B6
- net 3.3V: no longer U10.VCCA, U10.VCCA_2
- net D0_E: no longer U10.1A1
- net D10_E: no longer U10.2A3
- net D11_E: no longer U10.2A4
- net D1_E: no longer U10.1A2
- net D2_E: no longer U10.1A3
- net D3_E: no longer U10.1A4
- net D4_E: no longer U10.1A5
- net D5_E: no longer U10.1A6
- net D6_E: no longer U10.1A7
- net D7_E: no longer U10.1A8
- net D8_E: no longer U10.2A1
- net D9_E: no longer U10.2A2
- net FLASH: now also U$2.FLASH, U10.2B8; no longer TP7.TP, U0.13-FLASH
- net GND: now also U$2.AGND, U$2.DGND; no longer U0.2-DGND, U0.31-RSVR, U0.38-AGND, U0.39-AGND, U0.42-AGND, U0.43-AGND, U0.47-AGND, U0.5-DGND, U0.6-DGND, U10.GND, U10.GND_6, U10.GND_7, U10.GND_8
- net HSYNC_E: no longer U10.2A5
- net N$2: now also U$2.STANDBY; no longer U0.48-GND
- net OE_BAR_I: no longer U0.32-OE_BAR
- net OUTPUT_DRVR_EN: no longer R8.1, U10.!1OE, U10.!2OE
- net PIXCLK_E: no longer U10.2A7
- net RST_BAR_I: no longer U0.30-RESET_BAR
- net SADDR_I: no longer U0.10-SADDR
- net SCL_I: no longer U0.9-SCLK
- net SDA_I: no longer U0.14-SDATA
- net STANDBY_I: no longer U0.29-STANDBY
- net TRIG_I: no longer U0.33-TRIGGER
- net VAA: no longer C22.1, C4.1, U0.44-VAA, U0.45-VAA, U0.46-VAA
- net VAA_PIX: no longer C23.1, C5.1, U0.40-VAA_PIX, U0.41-VAA_PIX
- net VDD: no longer C1.1, C19.1, U0.3-VDD, U0.34-VDD, U0.4-VDD
- net VDD_IO: no longer C2.1, C20.1, U0.7-VDD_IO, U0.8-VDD_IO, U10.VCCB, U10.VCCB_2
- net VDD_PLL: no longer C21.1, C3.1, U0.1-VDD_PLL
- net VSYNC_E: no longer U10.2A6
Other:
- moved on the sheet: C1, C13, C14, C15, C19, C2, C20, C21, C22, C23, C27, C28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

Commit message: more schematic clean up
Parts:
- removed C33, C34, C35, C36, C37, C38: 1.0uF, SparkFun-Capacitors:1.0UF-0402-16V-10%
- added C10, C11, C12, C7, C8, C9: 1.0uF, SparkFun-Capacitors:1.0UF-0402-16V-10%
Connections:
- net FLASH renamed FLASH_I
- net HSYNC renamed HSYNC_I
- net PIXCLK renamed PIXCLK_I
- net VSYNC renamed VSYNC_I
- removed net D0_E: J2.3
- removed net D10_E: J2.13
- removed net D11_E: J2.14
- removed net D1_E: J2.4
- removed net D2_E: J2.5
- removed net D3_E: J2.6
- removed net D4_E: J2.7
- removed net D5_E: J2.8
- removed net D6_E: J2.9
- removed net D7_E: J2.10
- removed net D8_E: J2.11
- removed net D9_E: J2.12
- removed net N$10: U$2.OE_BAR
- removed net N$11: U$2.RESET_BAR
- removed net N$2: U$2.STANDBY
- removed net N$20: U13.A6
- removed net N$23: U13.A7
- removed net N$24: U13.A8
- removed net N$28: U13.B8
- removed net N$32: U13.B7
- removed net N$33: U13.B6
- removed net N$5: U$2.SADDR
- removed net N$6: U$2.SCLK
- removed net N$8: U$2.SDATA
- removed net N$9: U$2.TRIGGER
- removed net VAA: C36.1, TP6.TP, U15.OUT1
- removed net VAA_PIX: C37.1, TP5.TP, U15.OUT2
- removed net VDD: C33.1, TP1.TP, U12.OUT1
- removed net VDD_PLL: C35.1, TP2.TP, U14.OUT2
- new net DE_0: J2.3, U10.1A1
- new net DE_1: J2.4, U10.1A2
- new net DE_10: J2.13, U10.2A3
- new net DE_11: J2.14, U10.2A4
- new net DE_2: J2.5, U10.1A3
- new net DE_3: J2.6, U10.1A4
- new net DE_4: J2.7, U10.1A5
- new net DE_5: J2.8, U10.1A6
- new net DE_6: J2.9, U10.1A7
- new net DE_7: J2.10, U10.1A8
- new net DE_8: J2.11, U10.2A1
- new net DE_9: J2.12, U10.2A2
- new net FLASH_E: J2.35, U10.2A8
- net 1.8V: now also C7.1, TP2.TP, U12.OUT1
- net 2.8V: now also C25.1, C27.1, C30.1, C31.1, C6.2, C8.1, R10.1, R7.2, R9.2, TP4.TP, U13.VCCB, U13.VCCB_2, U14.OUT1, U9.VCCA
- net 3.3V: now also C12.1, TP1.TP, U10.VCCA, U10.VCCA_2; no longer C38.1, R9.2, TP3.TP
- net 5V: now also J2.38; no longer J2.35
- net DI_4: no longer U$2.DOUT5
- net DI_5: now also U$2.DOUT5
- net GND: now also C10.2, C11.2, C12.2, C7.2, C8.2, C9.2, U10.GND, U10.GND_6, U10.GND_7, U10.GND_8; no longer C33.2, C34.2, C35.2, C36.2, C37.2, C38.2, J2.38
- net HSYNC_E: now also U10.2A5
- net OE_BAR_I: now also U$2.OE_BAR
- net OUTPUT_DRVR_EN: now also R8.1, U10.!1OE, U10.!2OE
- net PIXCLK_E: now also U10.2A7
- net RST_BAR_I: now also U$2.RESET_BAR
- net SADDR_I: now also U$2.SADDR
- net SCL_I: now also U$2.SCLK
- net SDA_I: now also U$2.SDATA
- net STANDBY_I: now also U$2.STANDBY
- net TRIG_I: now also U$2.TRIGGER
- net VCC: now also C9.1, TP6.TP, U15.OUT1
- net VCC_1: now also C10.1, TP3.TP, U14.OUT2
- net VCC_2: now also C11.1, TP5.TP, U15.OUT2
- net VDD_IO: no longer C25.1, C27.1, C30.1, C31.1, C34.1, C6.2, R10.1, R7.2, TP4.TP, U13.VCCB, U13.VCCB_2, U14.OUT1, U9.VCCA
- net VSYNC_E: now also U10.2A6
Other:
- note added: "EXTCLK SELECT JUMPER"
- note added: "Optional I2C Pullup"
- note added: "VAA = 2.8V_2"
- note added: "VAA_PIX = 2.8V_4"
- note added: "VDD = 1.8V"
- note added: "VDD_IO = 2.8V_1"
- note added: "VDD_PLL = 2.8V_3"
- note removed: "Do I need a clock buffer here?"
- moved on the sheet: C1, C13, C14, C15, C19, C2, C20, C21, C22, C23, C24, C25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

Commit message: started rerouted board
Connections:
- removed net VDD_IO: U11.VCC
- net 2.8V: now also U11.VCC
- net 3.3V_EN: now also J2.30; no longer J2.28
- net CLK_EN: now also J2.21; no longer J2.34
- net EXTCLK: now also J2.20; no longer J2.18
- net FLASH_E: now also J2.18; no longer J2.35
- net INPUT_DRVR_EN: now also J2.29; no longer J2.27
- net OE_BAR_E: now also J2.23; no longer J2.20
- net OUTPUT_DRVR_EN: now also J2.19; no longer J2.26
- net RST_BAR_E: now also J2.24; no longer J2.21
- net SADDR_E: now also J2.26; no longer J2.23
- net SCL_E: now also J2.27; no longer J2.24
- net SDA_E: now also J2.28; no longer J2.25
- net STANDBY_E: now also J2.25; no longer J2.22
- net TRIG_E: now also J2.22; no longer J2.19
- net VAA_EN: now also J2.35; no longer J2.33
- net VAA_PIX_EN: now also J2.34; no longer J2.32
- net VDD18_EN: now also J2.31; no longer J2.29
- net VDD_IO_EN: now also J2.33; no longer J2.31
- net VDD_PLL_EN: now also J2.32; no longer J2.30

Commit message: finishing up board layout
Parts:
- JP1: value JUMPER-3SMD -> (none); device SparkFun-Passives:JUMPER-3SMD -> SparkFun-Passives:SOLDERJUMPER_2WAYPASTE1&2
Connections:
- new net EXTCLK_E: J2.20, JP1.3
- new net EXTCLK_I: JP1.1, U11.OUTPUT
- net 2.8V: now also C39.1, C40.1, U6.VDD, U7.A0, U7.VDD
- net 3.3V: no longer C39.1, C40.1, U6.VDD, U7.A0, U7.VDD
- net EXTCLK: no longer J2.20, JP1.1, JP1.3, U11.OUTPUT
Other:
- note added: "RIBBON CABLE"
- moved on the sheet: J2

Commit message: further refinement
Parts:
- JP1: value (none) -> CLKSEL
Other:
- note added: "EXTERNAL"
- note added: "IMAGE SENSOR"
Changed lines of the file:
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@@
 <setting verticaltext="up"/>
 </settings>
-<grid distance="0.05" unitdist="inch" unit="inch" style="lines" multiple="2" display="yes" altdistance="0.0125" altunitdist="inch" altunit="inch"/>
+<grid distance="1" unitdist="mm" unit="mm" style="lines" multiple="2" display="yes" altdistance="0.0125" altunitdist="inch" altunit="inch"/>
 <layers>
 <layer number="1" name="Top" color="4" fill="1" visible="no" active="no"/>
@@
 <part name="R11" library="SparkFun-Resistors" library_urn="urn:adsk.eagle:library:2058534" deviceset="RESISTOR" device="0402" package3d_urn="urn:adsk.eagle:package:2058625/2" value="10k"/>
 <part name="R12" library="SparkFun-Resistors" library_urn="urn:adsk.eagle:library:2058534" deviceset="RESISTOR" device="0402" package3d_urn="urn:adsk.eagle:package:2058625/2" value="10k"/>
-<part name="JP1" library="SparkFun-Passives" deviceset="SOLDERJUMPER_2WAY" device="PASTE1&amp;2"/>
+<part name="JP1" library="SparkFun-Passives" deviceset="SOLDERJUMPER_2WAY" device="PASTE1&amp;2" value="CLKSEL"/>
 <part name="GND1" library="SparkFun-PowerSymbols" deviceset="GND" device=""/>
 <part name="SUPPLY1" library="SparkFun-PowerSymbols" deviceset="1.8V" device=""/>
@@
 <wire x1="323.85" y1="215.9" x2="323.85" y2="168.91" width="0.508" layer="97"/>
 <wire x1="210.82" y1="168.91" x2="323.85" y2="168.91" width="0.508" layer="97"/>
+<text x="15" y="81" size="1.778" layer="97" rot="R90">IMAGE SENSOR</text>
+<text x="103" y="96" size="1.778" layer="97" rot="R270">EXTERNAL</text>
 </plain>
 <instances>
@@
 <instance part="R11" gate="G$1" x="215.9" y="31.75" rot="R90"/>
 <instance part="R12" gate="G$1" x="215.9" y="44.45" rot="R90"/>
-<instance part="JP1" gate="G$1" x="289.56" y="229.87" rot="R90"/>
+<instance part="JP1" gate="G$1" x="289.56" y="229.87" smashed="yes" rot="R90">
+<attribute name="NAME" x="291.465" y="234.3785" size="1.778" layer="95"/>
+<attribute name="VALUE" x="291.1475" y="232.41" size="1.778" layer="96"/>
+</instance>
 <instance part="GND1" gate="1" x="43.18" y="190.5"/>
 <instance part="SUPPLY1" gate="G$1" x="22.86" y="237.49"/>

Commit message: finishing touches!
Parts:
- R1: value 100 -> (none)
- R10, R11, R12, R2, R3, R4, R5, R6, R7, R8, R9: value 10k -> (none)
Other:
- moved on the sheet: C13, C14, C15, C24, C25, C27, C32, R10, R11, R12, R3, R4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
