File: oresat-camera-hardware/AR0130_DEV_BOARD/AR0130_DEV_BOARD_BREAKOUT.brd (EAGLE design)
At the start: 70 x 30 mm, 2 parts, among them J1 4-1734592-0

Commit message: finishing touches!
Routing:
- added copper zone on layer 16, net GND
Changed lines of the file:
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@@
 <setting verticaltext="up"/>
 </settings>
-<grid distance="0.25" unitdist="mm" unit="mm" style="lines" multiple="1" display="yes" altdistance="0.0625" altunitdist="mm" altunit="mm"/>
+<grid distance="2" unitdist="mm" unit="mm" style="lines" multiple="1" display="yes" altdistance="0.0125" altunitdist="mm" altunit="mm"/>
 <layers>
 <layer number="1" name="Top" color="4" fill="1" visible="yes" active="yes"/>
@@
 <vertex x="0" y="30"/>
 </polygon>
+<polygon width="0.2" layer="16">
+<vertex x="0" y="0"/>
+<vertex x="70" y="0"/>
+<vertex x="70" y="25.75"/>
+<vertex x="70" y="30"/>
+<vertex x="44.5" y="30"/>
+<vertex x="0" y="30"/>
+</polygon>
+<via x="10" y="10" extent="1-16" drill="0.35"/>
+<via x="6" y="2" extent="1-16" drill="0.35"/>
+<via x="8" y="2" extent="1-16" drill="0.35"/>
+<via x="10" y="2" extent="1-16" drill="0.35"/>
+<via x="12" y="2" extent="1-16" drill="0.35"/>
+<via x="14" y="2" extent="1-16" drill="0.35"/>
+<via x="16" y="2" extent="1-16" drill="0.35"/>
+<via x="18" y="2" extent="1-16" drill="0.35"/>
+<via x="20" y="2" extent="1-16" drill="0.35"/>
+<via x="22" y="2" extent="1-16" drill="0.35"/>
+<via x="24" y="2" extent="1-16" drill="0.35"/>
+<via x="26" y="2" extent="1-16" drill="0.35"/>
+<via x="28" y="2" extent="1-16" drill="0.35"/>
+<via x="30" y="2" extent="1-16" drill="0.35"/>
+<via x="32" y="2" extent="1-16" drill="0.35"/>
+<via x="34" y="2" extent="1-16" drill="0.35"/>
+<via x="36" y="2" extent="1-16" drill="0.35"/>
+<via x="38" y="2" extent="1-16" drill="0.35"/>
+<via x="40" y="2" extent="1-16" drill="0.35"/>
+<via x="42" y="2" extent="1-16" drill="0.35"/>
+<via x="44" y="2" extent="1-16" drill="0.35"/>
+<via x="46" y="2" extent="1-16" drill="0.35"/>
+<via x="48" y="2" extent="1-16" drill="0.35"/>
+<via x="50" y="2" extent="1-16" drill="0.35"/>
+<via x="52" y="2" extent="1-16" drill="0.35"/>
+<via x="54" y="2" extent="1-16" drill="0.35"/>
+<via x="56" y="2" extent="1-16" drill="0.35"/>
+<via x="58" y="2" extent="1-16" drill="0.35"/>
+<via x="60" y="2" extent="1-16" drill="0.35"/>
+<via x="62" y="2" extent="1-16" drill="0.35"/>
+<via x="64" y="2" extent="1-16" drill="0.35"/>
+<via x="68" y="6" extent="1-16" drill="0.35"/>
+<via x="68" y="8" extent="1-16" drill="0.35"/>
+<via x="68" y="10" extent="1-16" drill="0.35"/>
+<via x="68" y="12" extent="1-16" drill="0.35"/>
+<via x="68" y="14" extent="1-16" drill="0.35"/>
+<via x="68" y="16" extent="1-16" drill="0.35"/>
+<via x="68" y="18" extent="1-16" drill="0.35"/>
+<via x="68" y="20" extent="1-16" drill="0.35"/>
+<via x="68" y="22" extent="1-16" drill="0.35"/>
+<via x="2" y="6" extent="1-16" drill="0.35"/>
+<via x="2" y="8" extent="1-16" drill="0.35"/>
+<via x="2" y="10" extent="1-16" drill="0.35"/>
+<via x="2" y="12" extent="1-16" drill="0.35"/>
+<via x="2" y="14" extent="1-16" drill="0.35"/>
+<via x="2" y="16" extent="1-16" drill="0.35"/>
+<via x="2" y="18" extent="1-16" drill="0.35"/>
+<via x="2" y="20" extent="1-16" drill="0.35"/>
+<via x="2" y="22" extent="1-16" drill="0.35"/>
+<via x="2" y="24" extent="1-16" drill="0.35"/>
+<via x="6" y="28" extent="1-16" drill="0.35"/>
+<via x="8" y="28" extent="1-16" drill="0.35"/>
+<via x="10" y="28" extent="1-16" drill="0.35"/>
+<via x="12" y="28" extent="1-16" drill="0.35"/>
+<via x="14" y="28" extent="1-16" drill="0.35"/>
+<via x="16" y="28" extent="1-16" drill="0.35"/>
+<via x="18" y="28" extent="1-16" drill="0.35"/>
+<via x="20" y="28" extent="1-16" drill="0.35"/>
+<via x="22" y="28" extent="1-16" drill="0.35"/>
+<via x="24" y="28" extent="1-16" drill="0.35"/>
+<via x="26" y="28" extent="1-16" drill="0.35"/>
+<via x="28" y="28" extent="1-16" drill="0.35"/>
+<via x="30" y="28" extent="1-16" drill="0.35"/>
+<via x="48" y="28" extent="1-16" drill="0.35"/>
+<via x="50" y="28" extent="1-16" drill="0.35"/>
+<via x="52" y="28" extent="1-16" drill="0.35"/>
+<via x="54" y="28" extent="1-16" drill="0.35"/>
+<via x="56" y="28" extent="1-16" drill="0.35"/>
+<via x="58" y="28" extent="1-16" drill="0.35"/>
+<via x="60" y="28" extent="1-16" drill="0.35"/>
+<via x="62" y="28" extent="1-16" drill="0.35"/>
+<via x="64" y="28" extent="1-16" drill="0.35"/>
+<via x="8" y="24" extent="1-16" drill="0.35"/>
+<via x="12" y="24" extent="1-16" drill="0.35"/>
+<via x="16" y="24" extent="1-16" drill="0.35"/>
+<via x="20" y="24" extent="1-16" drill="0.35"/>
+<via x="20" y="20" extent="1-16" drill="0.35"/>
+<via x="16" y="20" extent="1-16" drill="0.35"/>
+<via x="12" y="20" extent="1-16" drill="0.35"/>
+<via x="8" y="20" extent="1-16" drill="0.35"/>
+<via x="8" y="16" extent="1-16" drill="0.35"/>
+<via x="12" y="16" extent="1-16" drill="0.35"/>
+<via x="16" y="16" extent="1-16" drill="0.35"/>
+<via x="4" y="16" extent="1-16" drill="0.35"/>
+<via x="4" y="20" extent="1-16" drill="0.35"/>
+<via x="4" y="24" extent="1-16" drill="0.35"/>
+<via x="4" y="12" extent="1-16" drill="0.35"/>
+<via x="8" y="12" extent="1-16" drill="0.35"/>
+<via x="8" y="8" extent="1-16" drill="0.35"/>
+<via x="4" y="8" extent="1-16" drill="0.35"/>
+<via x="8" y="4" extent="1-16" drill="0.35"/>
+<via x="12" y="4" extent="1-16" drill="0.35"/>
+<via x="16" y="4" extent="1-16" drill="0.35"/>
+<via x="20" y="4" extent="1-16" drill="0.35"/>
+<via x="24" y="4" extent="1-16" drill="0.35"/>
+<via x="28" y="4" extent="1-16" drill="0.35"/>
+<via x="32" y="4" extent="1-16" drill="0.35"/>
+<via x="36" y="4" extent="1-16" drill="0.35"/>
+<via x="40" y="4" extent="1-16" drill="0.35"/>
+<via x="44" y="4" extent="1-16" drill="0.35"/>
+<via x="48" y="4" extent="1-16" drill="0.35"/>
+<via x="52" y="4" extent="1-16" drill="0.35"/>
+<via x="56" y="4" extent="1-16" drill="0.35"/>
+<via x="60" y="4" extent="1-16" drill="0.35"/>
+<via x="64" y="4" extent="1-16" drill="0.35"/>
+<via x="64" y="8" extent="1-16" drill="0.35"/>
+<via x="64" y="12" extent="1-16" drill="0.35"/>
+<via x="64" y="16" extent="1-16" drill="0.35"/>
+<via x="60" y="16" extent="1-16" drill="0.35"/>
+<via x="60" y="20" extent="1-16" drill="0.35"/>
+<via x="64" y="20" extent="1-16" drill="0.35"/>
+<via x="64" y="24" extent="1-16" drill="0.35"/>
+<via x="60" y="24" extent="1-16" drill="0.35"/>
+<via x="68" y="24" extent="1-16" drill="0.35"/>
+<via x="56" y="24" extent="1-16" drill="0.35"/>
+<via x="56" y="20" extent="1-16" drill="0.35"/>
+<via x="52" y="20" extent="1-16" drill="0.35"/>
+<via x="52" y="24" extent="1-16" drill="0.35"/>
+<via x="48" y="24" extent="1-16" drill="0.35"/>
+<via x="22.4" y="15.225" extent="1-16" drill="0.35"/>
+<via x="19.6125" y="13.5625" extent="1-16" drill="0.35"/>
+<via x="24.875" y="17.1" extent="1-16" drill="0.35"/>
+<via x="31.7125" y="17.0125" extent="1-16" drill="0.35"/>
+<via x="33.65" y="15.1875" extent="1-16" drill="0.35"/>
+<via x="36.2125" y="12.8375" extent="1-16" drill="0.35"/>
+<via x="31.15" y="15.1375" extent="1-16" drill="0.35"/>
+<via x="41.45" y="19.35" extent="1-16" drill="0.35"/>
+<via x="43.8625" y="18.6" extent="1-16" drill="0.35"/>
+<via x="46.4375" y="14.825" extent="1-16" drill="0.35"/>
+<via x="49.0875" y="14.9875" extent="1-16" drill="0.35"/>
+<via x="53.8375" y="12.9125" extent="1-16" drill="0.35"/>
+<via x="51.4375" y="12.825" extent="1-16" drill="0.35"/>
+<via x="43.7875" y="12.8125" extent="1-16" drill="0.35"/>
+<via x="41.4" y="12.65" extent="1-16" drill="0.35"/>
+<via x="38.6125" y="20.375" extent="1-16" drill="0.35"/>
+<via x="29.0875" y="14.5875" extent="1-16" drill="0.35"/>
+<via x="26.8375" y="13.7375" extent="1-16" drill="0.35"/>
+<via x="24.225" y="12.9" extent="1-16" drill="0.35"/>
+<via x="12" y="6" extent="1-16" drill="0.35"/>
+<via x="20" y="6" extent="1-16" drill="0.35"/>
+<via x="28" y="6" extent="1-16" drill="0.35"/>
+<via x="36" y="6" extent="1-16" drill="0.35"/>
+<via x="44" y="6" extent="1-16" drill="0.35"/>
+<via x="52" y="6" extent="1-16" drill="0.35"/>
+<via x="60" y="6" extent="1-16" drill="0.35"/>
 </signal>
 <signal name="D0">

Commit message: more final touches on bouard
Changed lines of the file:
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@@
 <via x="22" y="2" extent="1-16" drill="0.35"/>
 <via x="24" y="2" extent="1-16" drill="0.35"/>
-<via x="26" y="2" extent="1-16" drill="0.35"/>
+<via x="26" y="1.5" extent="1-16" drill="0.35"/>
 <via x="28" y="2" extent="1-16" drill="0.35"/>
 <via x="30" y="2" extent="1-16" drill="0.35"/>
@@
 <via x="8" y="16" extent="1-16" drill="0.35"/>
 <via x="12" y="16" extent="1-16" drill="0.35"/>
-<via x="16" y="16" extent="1-16" drill="0.35"/>
+<via x="17" y="16" extent="1-16" drill="0.35"/>
 <via x="4" y="16" extent="1-16" drill="0.35"/>
 <via x="4" y="20" extent="1-16" drill="0.35"/>
@@
 <via x="16" y="4" extent="1-16" drill="0.35"/>
 <via x="20" y="4" extent="1-16" drill="0.35"/>
-<via x="24" y="4" extent="1-16" drill="0.35"/>
+<via x="24.5" y="4" extent="1-16" drill="0.35"/>
 <via x="28" y="4" extent="1-16" drill="0.35"/>
 <via x="32" y="4" extent="1-16" drill="0.35"/>
@@
 <via x="19.6125" y="13.5625" extent="1-16" drill="0.35"/>
 <via x="24.875" y="17.1" extent="1-16" drill="0.35"/>
-<via x="31.7125" y="17.0125" extent="1-16" drill="0.35"/>
-<via x="33.65" y="15.1875" extent="1-16" drill="0.35"/>
+<via x="31.775" y="16.7375" extent="1-16" drill="0.35"/>
+<via x="34.2125" y="14.8125" extent="1-16" drill="0.35"/>
 <via x="36.2125" y="12.8375" extent="1-16" drill="0.35"/>
-<via x="31.15" y="15.1375" extent="1-16" drill="0.35"/>
-<via x="41.45" y="19.35" extent="1-16" drill="0.35"/>
+<via x="30.5875" y="15.8375" extent="1-16" drill="0.35"/>
+<via x="41.3375" y="19.6625" extent="1-16" drill="0.35"/>
 <via x="43.8625" y="18.6" extent="1-16" drill="0.35"/>
-<via x="46.4375" y="14.825" extent="1-16" drill="0.35"/>
-<via x="49.0875" y="14.9875" extent="1-16" drill="0.35"/>
+<via x="46.35" y="14.775" extent="1-16" drill="0.35"/>
+<via x="48.95" y="15.4" extent="1-16" drill="0.35"/>
 <via x="53.8375" y="12.9125" extent="1-16" drill="0.35"/>
 <via x="51.4375" y="12.825" extent="1-16" drill="0.35"/>
 <via x="43.7875" y="12.8125" extent="1-16" drill="0.35"/>
 <via x="41.4" y="12.65" extent="1-16" drill="0.35"/>
-<via x="38.6125" y="20.375" extent="1-16" drill="0.35"/>
-<via x="29.0875" y="14.5875" extent="1-16" drill="0.35"/>
-<via x="26.8375" y="13.7375" extent="1-16" drill="0.35"/>
+<via x="38.9125" y="21.1625" extent="1-16" drill="0.35"/>
+<via x="29.2" y="14.7" extent="1-16" drill="0.35"/>
+<via x="26.7625" y="13.725" extent="1-16" drill="0.35"/>
 <via x="24.225" y="12.9" extent="1-16" drill="0.35"/>
 <via x="12" y="6" extent="1-16" drill="0.35"/>
 <via x="20" y="6" extent="1-16" drill="0.35"/>
 <via x="28" y="6" extent="1-16" drill="0.35"/>
-<via x="36" y="6" extent="1-16" drill="0.35"/>
-<via x="44" y="6" extent="1-16" drill="0.35"/>
+<via x="35.5" y="6" extent="1-16" drill="0.35"/>
+<via x="44.5" y="6" extent="1-16" drill="0.35"/>
 <via x="52" y="6" extent="1-16" drill="0.35"/>
 <via x="60" y="6" extent="1-16" drill="0.35"/>

Commit message: yada yada yada
Connections:
- net 5V: now also U$1.34, U$1.36; no longer U$1.37, U$1.39
- net GND: now also U$1.37, U$1.39; no longer U$1.34, U$1.36
