File: oresat-camera-hardware/AR0130_DEV_BOARD/AR0130_DEV_BOARD_BREAKOUT.sch (EAGLE design)
At the start: 2 parts, among them J1 4-1734592-0

Commit message: further refinement
Changed lines of the file:
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@@
 <segment>
 <pinref part="U$1" gate="A" pin="32"/>
-<wire x1="38.1" y1="-15.24" x2="43.18" y2="-7.62" width="0.1524" layer="91"/>
-<label x="43.18" y="-7.62" size="1.27" layer="95" rot="R90" xref="yes"/>
+<wire x1="38.1" y1="-15.24" x2="38.18" y2="-7.62" width="0.1524" layer="91"/>
+<label x="38.18" y="-7.62" size="1.27" layer="95" rot="R90" xref="yes"/>
 </segment>
 </net>
@@
 <segment>
 <pinref part="U$1" gate="A" pin="28"/>
-<wire x1="43.18" y1="-15.24" x2="38.1" y2="-7.62" width="0.1524" layer="91"/>
-<label x="38.1" y="-7.62" size="1.27" layer="95" rot="R90" xref="yes"/>
+<wire x1="43.18" y1="-15.24" x2="43.1" y2="-7.62" width="0.1524" layer="91"/>
+<label x="43.1" y="-7.62" size="1.27" layer="95" rot="R90" xref="yes"/>
 </segment>
 </net>

Commit message: finishing touches!
Other:
- note added: "40x2 HEADER"
- note added: "RIBBON CABLE"
- moved on the sheet: J1, U$1

Commit message: yada yada yada
Connections:
- net 5V: now also U$1.34, U$1.36; no longer U$1.37, U$1.39
- net GND: now also U$1.37, U$1.39; no longer U$1.34, U$1.36
Changed lines of the file:
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@@
 <part name="SUPPLY2" library="SparkFun-PowerSymbols" deviceset="5V" device=""/>
 <part name="SUPPLY3" library="SparkFun-PowerSymbols" deviceset="5V" device=""/>
-<part name="SUPPLY4" library="SparkFun-PowerSymbols" deviceset="5V" device=""/>
-<part name="SUPPLY5" library="SparkFun-PowerSymbols" deviceset="5V" device=""/>
 <part name="GND5" library="SparkFun-PowerSymbols" deviceset="GND" device=""/>
 <part name="GND6" library="SparkFun-PowerSymbols" deviceset="GND" device=""/>
 <part name="SUPPLY6" library="SparkFun-PowerSymbols" deviceset="5V" device=""/>
+<part name="FRAME1" library="frames" library_urn="urn:adsk.eagle:library:229" deviceset="A5L-LOC" device=""/>
+<part name="SUPPLY7" library="SparkFun-PowerSymbols" deviceset="5V" device=""/>
+<part name="SUPPLY8" library="SparkFun-PowerSymbols" deviceset="5V" device=""/>
 <part name="GND7" library="SparkFun-PowerSymbols" deviceset="GND" device=""/>
 <part name="GND8" library="SparkFun-PowerSymbols" deviceset="GND" device=""/>
-<part name="FRAME1" library="frames" library_urn="urn:adsk.eagle:library:229" deviceset="A5L-LOC" device=""/>
 </parts>
 <sheets>
@@
 <attribute name="VALUE" x="75.438" y="89.154" size="1.778" layer="96" rot="R270" align="bottom-center"/>
 </instance>
-<instance part="SUPPLY4" gate="G$1" x="17.78" y="25.4" smashed="yes" rot="R180">
-<attribute name="VALUE" x="17.018" y="20.574" size="1.778" layer="96" rot="R270" align="bottom-center"/>
-</instance>
-<instance part="SUPPLY5" gate="G$1" x="15.24" y="25.4" smashed="yes" rot="R180">
-<attribute name="VALUE" x="14.478" y="20.574" size="1.778" layer="96" rot="R270" align="bottom-center"/>
-</instance>
 <instance part="GND5" gate="1" x="17.78" y="71.12" smashed="yes" rot="R180">
 <attribute name="VALUE" x="18.542" y="74.422" size="1.778" layer="96" rot="R270" align="top-center"/>
@@
 <attribute name="VALUE" x="19.558" y="20.574" size="1.778" layer="96" rot="R270" align="bottom-center"/>
 </instance>
-<instance part="GND7" gate="1" x="20.32" y="71.12" smashed="yes" rot="R180">
-<attribute name="VALUE" x="21.082" y="74.422" size="1.778" layer="96" rot="R270" align="top-center"/>
-</instance>
-<instance part="GND8" gate="1" x="22.86" y="71.12" smashed="yes" rot="R180">
-<attribute name="VALUE" x="23.622" y="74.422" size="1.778" layer="96" rot="R270" align="top-center"/>
-</instance>
 <instance part="FRAME1" gate="G$1" x="0" y="0"/>
+<instance part="SUPPLY7" gate="G$1" x="22.86" y="68.58" smashed="yes">
+<attribute name="VALUE" x="23.622" y="73.406" size="1.778" layer="96" rot="R90" align="bottom-center"/>
+</instance>
+<instance part="SUPPLY8" gate="G$1" x="20.32" y="68.58" smashed="yes">
+<attribute name="VALUE" x="21.082" y="73.406" size="1.778" layer="96" rot="R90" align="bottom-center"/>
+</instance>
+<instance part="GND7" gate="1" x="17.78" y="22.86" smashed="yes">
+<attribute name="VALUE" x="17.018" y="19.558" size="1.778" layer="96" rot="R90" align="top-center"/>
+</instance>
+<instance part="GND8" gate="1" x="15.24" y="22.86" smashed="yes">
+<attribute name="VALUE" x="14.478" y="19.558" size="1.778" layer="96" rot="R90" align="top-center"/>
+</instance>
 </instances>
 <busses>
@@
 </segment>
 <segment>
-<pinref part="U$1" gate="A" pin="34"/>
-<wire x1="22.86" y1="60.96" x2="22.86" y2="68.58" width="0.1524" layer="91"/>
+<pinref part="U$1" gate="A" pin="39"/>
+<wire x1="15.24" y1="33.02" x2="15.24" y2="25.4" width="0.1524" layer="91"/>
 <pinref part="GND8" gate="1" pin="GND"/>
 </segment>
 <segment>
-<pinref part="U$1" gate="A" pin="36"/>
-<wire x1="20.32" y1="60.96" x2="20.32" y2="68.58" width="0.1524" layer="91"/>
+<pinref part="U$1" gate="A" pin="37"/>
+<wire x1="17.78" y1="33.02" x2="17.78" y2="25.4" width="0.1524" layer="91"/>
 <pinref part="GND7" gate="1" pin="GND"/>
 </segment>
@@
 </segment>
 <segment>
-<pinref part="U$1" gate="A" pin="37"/>
-<wire x1="17.78" y1="33.02" x2="17.78" y2="25.4" width="0.1524" layer="91"/>
-<pinref part="SUPPLY4" gate="G$1" pin="5V"/>
-</segment>
-<segment>
-<pinref part="U$1" gate="A" pin="39"/>
-<wire x1="15.24" y1="33.02" x2="15.24" y2="25.4" width="0.1524" layer="91"/>
-<pinref part="SUPPLY5" gate="G$1" pin="5V"/>
-</segment>
-<segment>
 <pinref part="U$1" gate="A" pin="35"/>
 <wire x1="20.32" y1="33.02" x2="20.32" y2="25.4" width="0.1524" layer="91"/>
 <pinref part="SUPPLY6" gate="G$1" pin="5V"/>
 </segment>
-</net>
+<segment>
+<pinref part="U$1" gate="A" pin="34"/>
+<wire x1="22.86" y1="60.96" x2="22.86" y2="68.58" width="0.1524" layer="91"/>
+<pinref part="SUPPLY7" gate="G$1" pin="5V"/>
+</segment>
+<segment>
+<pinref part="U$1" gate="A" pin="36"/>
+<wire x1="20.32" y1="60.96" x2="20.32" y2="68.58" width="0.1524" layer="91"/>
+<pinref part="SUPPLY8" gate="G$1" pin="5V"/>
+</segment>
+</net>
