File: oresat-camera-hardware/AR0130_DEV_BOARD/ARCHIVE/AR0130_DEV_BOARD_SCHEMATIC_V1.sch (EAGLE design)
At the start: 84 parts, among them J2 4-1734592-04-1734592-0, U10 SN74AVCB164245VR, U11 KC2520B27.0000C10E00, U12 TPS71818-33DRVT, U13 SN74AVCH8T245RHLR, U14 TPS71928-28DRVT, U15 TPS71928-28DRVT, U6 MCP9808T-E/MCDFN8_2X3MC-M, U7 MCP9808T-E/MCDFN8_2X3MC-M, U9 TCA9509DGKRDGK8-M

Commit message: EVERYTHING IS FINE. Updated board for totally correct footprint this time I swear
Parts:
- removed TP14, TP15, TP16, TP17, TP18, TP19, TP20, TP21, TP22, TP23, TP24, TP25, TP26, TP27, TP28: TPTP06R, testpad:TPTP06R
- J2: value 4-1734592-04-1734592-0 -> 4-1734592-0; device Oliver_Custom:4-1734592-04-1734592-0 -> Oliver_Custom:4-1734592-0
- U$2: value AR0130CSSM00SPCA0−DRBR1-847AC-ILCC -> AR0130CSSM00SPCA0−DRBR1-847AB; device Oliver_Custom:AR0130CSSM00SPCA0−DRBR1-847AC-ILCC -> Oliver_Custom:AR0130CSSM00SPCA0−DRBR1-847AB
Connections:
- net 3.3V_EN: now also J2.30; no longer J2.8
- net CLK_EN: now also J2.21; no longer J2.27
- net DE_0: now also J2.3, U10.1A1; no longer J2.21, U10.2A5
- net DE_1: now also J2.4, U10.1A2; no longer J2.20, U10.2A4
- net DE_10: now also J2.13, U10.2A3; no longer J2.11, U10.1A3
- net DE_11: now also J2.14, U10.2A4; no longer J2.10, U10.1A2
- net DE_2: now also J2.5, U10.1A3; no longer J2.19, U10.2A3
- net DE_3: now also J2.6, U10.1A4; no longer J2.18, U10.2A2
- net DE_4: now also J2.7, U10.1A5; no longer J2.17, U10.2A1
- net DE_5: now also J2.8, U10.1A6; no longer J2.16, U10.1A8
- net DE_6: now also J2.9; no longer J2.15
- net DE_7: now also J2.10, U10.1A8; no longer J2.14, U10.1A6
- net DE_8: now also J2.11, U10.2A1; no longer J2.13, U10.1A5
- net DE_9: now also U10.2A2; no longer U10.1A4
- net DI_0: now also U10.1B1; no longer TP14.TP, U10.2B5
- net DI_1: now also U10.1B2; no longer TP15.TP, U10.2B4
- net DI_10: now also U10.2B3; no longer TP24.TP, U10.1B3
- net DI_11: now also U10.2B4; no longer TP25.TP, U10.1B2
- net DI_2: now also U10.1B3; no longer TP16.TP, U10.2B3
- net DI_3: now also U10.1B4; no longer TP17.TP, U10.2B2
- net DI_4: now also U10.1B5; no longer TP18.TP, U10.2B1
- net DI_5: now also U10.1B6; no longer TP19.TP, U10.1B8
- net DI_6: no longer TP20.TP
- net DI_7: now also U10.1B8; no longer TP21.TP, U10.1B6
- net DI_8: now also U10.2B1; no longer TP22.TP, U10.1B5
- net DI_9: now also U10.2B2; no longer TP23.TP, U10.1B4
- net EXTCLK_E: now also J2.20; no longer J2.26
- net FLASH_E: now also J2.18; no longer J2.24
- net GND: no longer J2.PAD
- net HSYNC_E: now also J2.15, U10.2A5; no longer J2.23, U10.2A7
- net HSYNC_I: now also U10.2B5; no longer TP26.TP, U10.2B7
- net INPUT_DRVR_EN: now also J2.29; no longer J2.33
- net OE_BAR_E: now also J2.23, U13.A4; no longer J2.30, U13.A3
- net OE_BAR_I: now also U13.B4; no longer U13.B3
- net OUTPUT_DRVR_EN: now also J2.19; no longer J2.25
- net PIXCLK_E: now also J2.17, U10.2A7; no longer J2.9, U10.1A1
- net PIXCLK_I: now also U10.2B7; no longer TP28.TP, U10.1B1
- net RST_BAR_E: now also J2.24, U13.A3; no longer J2.28, U13.A5
- net RST_BAR_I: now also U13.B3; no longer U13.B5
- net SADDR_E: now also J2.26, U13.A1; no longer J2.31, U13.A2
- net SADDR_I: now also U13.B1; no longer U13.B2
- net SCL_E: now also J2.27; no longer J2.34
- net SDA_E: now also J2.28; no longer J2.35
- net STANDBY_E: now also J2.25, U13.A2; no longer J2.29, U13.A4
- net STANDBY_I: now also U13.B2; no longer U13.B4
- net TRIG_E: now also J2.22, U13.A5; no longer J2.32, U13.A1
- net TRIG_I: now also U13.B5; no longer U13.B1
- net VAA_EN: now also J2.35; no longer J2.3
- net VAA_PIX_EN: now also J2.34; no longer J2.4
- net VDD18_EN: now also J2.31; no longer J2.7
- net VDD_IO_EN: now also J2.33; no longer J2.5
- net VDD_PLL_EN: now also J2.32; no longer J2.6
- net VSYNC_E: now also J2.16; no longer J2.22
- net VSYNC_I: no longer TP27.TP
Other:
- moved on the sheet: C6, JP1, R2, R5, R6, R8, TP10, TP11, TP7, TP8, TP9, U10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
