File: oresat-camera-hardware/AR0130_DEV_BOARD/REV3/AR0130_DEV_BOARD.sch (EAGLE design)
At the start: 84 parts, among them J2 4-1734592-04-1734592-0, U1 SN74AVCB164245VR, U11 KC2520B27.0000C10E00, U13 SN74AVCH8T245RHLR, U2 TPS71928-28DRVT, U3 TPS71928-28DRVT, U4 TPS71818-33DRVT, U6 MCP9808T-E/MCDFN8_2X3MC-M, U7 MCP9808T-E/MCDFN8_2X3MC-M, U9 TCA9509DGKRDGK8-M

Commit message: addressed some camera board revisions for 3rd rev
Parts:
- removed U1: SN74AVCB164245VR, Oliver_Custom:SN74AVCB164245VR
- removed U2, U3: TPS71928-28DRVT, Oliver_Custom:TPS71928-28DRVT
- removed U4: TPS71818-33DRVT, Oliver_Custom:TPS71818-33DRVT
- added U10: SN74AVCB164245VR, Oliver_Custom:SN74AVCB164245VR
- added U12: TPS71818-33DRVT, Oliver_Custom:TPS71818-33DRVT
- added U14, U15: TPS71928-28DRVT, Oliver_Custom:TPS71928-28DRVT
Connections:
- net 1.8V: now also U12.OUT1
- net 2.8V: now also U10.VCCB, U10.VCCB_2, U14.OUT1, U6.A0, U6.A1; no longer U1.VCCB
- net 3.3V: now also U10.VCCA, U10.VCCA_2, U12.OUT2; no longer U1.VCCA
- net 3.3V_EN: now also U12.EN2
- net 5V: now also U12.IN, U14.IN, U15.IN; no longer U2.VIN
- net DE_0: now also U10.2A5; no longer U1.2A5
- net DE_1: now also U10.2A4; no longer U1.2A4
- net DE_10: now also U10.1A3; no longer U1.1A3
- net DE_11: now also U10.1A2; no longer U1.1A2
- net DE_2: now also U10.2A3; no longer U1.2A3
- net DE_3: now also U10.2A2; no longer U1.2A2
- net DE_4: now also U10.2A1; no longer U1.2A1
- net DE_5: now also U10.1A8; no longer U1.1A8
- net DE_6: now also U10.1A7; no longer U1.1A7
- net DE_7: now also U10.1A6; no longer U1.1A6
- net DE_8: now also U10.1A5; no longer U1.1A5
- net DE_9: now also U10.1A4; no longer U1.1A4
- net DI_0: now also U10.2B5; no longer U1.2B5
- net DI_1: now also U10.2B4; no longer U1.2B4
- net DI_10: now also U10.1B3; no longer U1.1B3
- net DI_11: now also U10.1B2; no longer U1.1B2
- net DI_2: now also U10.2B3; no longer U1.2B3
- net DI_3: now also U10.2B2; no longer U1.2B2
- net DI_4: now also U10.2B1; no longer U1.2B1
- net DI_5: now also U10.1B8; no longer U1.1B8
- net DI_6: now also U10.1B7; no longer U1.1B7
- net DI_7: now also U10.1B6; no longer U1.1B6
- net DI_8: now also U10.1B5; no longer U1.1B5
- net DI_9: now also U10.1B4; no longer U1.1B4
- net FLASH_E: now also U10.2A8; no longer U1.2A8
- net FLASH_I: now also U10.2B8; no longer U1.2B8
- net GND: now also U10.GND, U10.GND_2, U10.GND_3, U10.GND_4, U10.GND_5, U10.GND_6, U10.GND_7, U10.GND_8, U12.EPAD, U12.GND, U14.EPAD, U14.GND, U15.EPAD, U15.GND; no longer U1.GND, U2.GND, U3.GND, U6.A0, U6.A1
- net HSYNC_E: now also U10.2A7; no longer U1.2A7
- net HSYNC_I: now also U10.2B7; no longer U1.2B7
- net N$25: now also U10.2DIR; no longer U1.2DIR
- net N$3: now also U10.1DIR; no longer U1.1DIR
- net OUTPUT_DRVR_EN: now also U10.!1OE, U10.!2OE; no longer U1.!1OE, U1.!2OE
- net PIXCLK_E: now also U10.1A1; no longer U1.1A1
- net PIXCLK_I: now also U10.1B1; no longer U1.1B1
- net VAA_EN: now also U15.EN1; no longer U2.EN1
- net VAA_PIX_EN: now also U15.EN2; no longer U2.EN2
- net VCC: now also U15.OUT1; no longer U2.OUT1
- net VCC_1: now also U14.OUT2
- net VCC_2: now also U15.OUT2; no longer U2.OUT2
- net VDD18_EN: now also U12.EN1
- net VDD_IO_EN: now also U14.EN1
- net VDD_PLL_EN: now also U14.EN2
- net VSYNC_E: now also U10.2A6; no longer U1.2A6
- net VSYNC_I: now also U10.2B6; no longer U1.2B6
Other:
- note added: "I2C ADDR: 0x19"
- note added: "I2C ADDR: 0x1B"
- note removed: "I2C ADDR:"
- moved on the sheet: C39, C40, R5, R6, R8, TP1, TP2, TP3, TP4, TP5, TP6, U6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
