File: oresat-camera-hardware/oresat-camera-board/AR0130_DEV_BOARD.brd (EAGLE design)
At the start: 31.5 x 14 mm, 42 parts, among them J1 4-1734742-0, U1 TPS71928-28DRVT, U2 TPS71928-28DRVT, U3 TPS70618DRVR, U4 AR0134CSSM00SPCA0, X1 KC2520B27.0000C10E00

Commit message: some final touchs, think it's ready for review
Parts:
- removed C20, C21, C22: 0.1uF, oresat-rcl:.0402-B-NOSILK
- removed TP11, TP29: TPTP06R, J-TestPoint-Small:TP06R
- removed U$1: (no value), Oliver_Custom:M12-LENS-MOUNT
- added C15, C18: 2.2uF, oresat-rcl:.0603-C-NOSILK
- added C16: 10uF, oresat-rcl:.0603-C-NOSILK
- added TP6, TP7: TPTP06R, J-TestPoint-Small:TP06R
- C1: value 10uF -> 10nF; device oresat-rcl:.0603-C-NOSILK -> oresat-rcl:.0402-A-NOSILK
- C10: value 2.2uF -> 1.0uF
- C12: value 1.0uF -> 10uF
- C13: value 1.0uF -> 0.1uF; device oresat-rcl:.0603-C-NOSILK -> oresat-rcl:.0402-B-NOSILK
- C19: value 0.1uF -> 2.2uF; device oresat-rcl:.0402-B-NOSILK -> oresat-rcl:.0603-C-NOSILK
- C3, C5: value 10uF -> 0.1uF; device oresat-rcl:.0603-C-NOSILK -> oresat-rcl:.0402-B-NOSILK
- C6: value 10nF -> 1.0uF; device oresat-rcl:.0402-A-NOSILK -> oresat-rcl:.0603-C-NOSILK
- C8: value 2.2uF -> 10uF
- C9: value 2.2uF -> 0.1uF; device oresat-rcl:.0603-C-NOSILK -> oresat-rcl:.0402-B-NOSILK
- R1: value 100 -> 10k
- R2: value 10k -> 100
- R3: value 10K -> 10k
- R4: value DNP -> 10k
- R5: value 10k -> 10K
- R6: value 10k -> DNP
- U1: value TPS71928-28DRVT -> AR0134CSSM00SPCA0; device U-TI-TPS71928-28-VoltageReg:DRV6_1P6X1 -> U-ONSemi-AR0134:AR0134CSSM00SPCA0
- U2: value TPS71928-28DRVT -> TPS70618DRVR; device U-TI-TPS71928-28-VoltageReg:DRV6_1P6X1 -> U-TI-TPS70618-VoltageReg:DRV6_1P6X1
- U3: value TPS70618DRVR -> TPS71928-28DRVT; device U-TI-TPS70618-VoltageReg:DRV6_1P6X1 -> U-TI-TPS71928-28-VoltageReg:DRV6_1P6X1
- U4: value AR0134CSSM00SPCA0 -> TPS71928-28DRVT; device U-ONSemi-AR0134:AR0134CSSM00SPCA0 -> U-TI-TPS71928-28-VoltageReg:DRV6_1P6X1
- moved TP2 24.5 mm to (29.2, 1.50)
- moved TP3 24.5 mm to (28.5, 2.25)
- moved R3 24.3 mm to (0.75, 8.50), turned to 270 degrees
- moved R5 24.3 mm to (25.0, 7.75), turned to 90 degrees
- moved TP10 23.6 mm to (5.75, 4.00)
- moved R4 23.2 mm to (0.75, 10.5)
- moved R6 23.2 mm to (23.8, 7.75)
- moved TP1 22.4 mm to (27.8, 1.50)
- moved U4 17.7 mm to (24.5, 4.25), flipped to the bottom, turned to 90 degrees
- moved C6 16.0 mm to (20.0, 1.62)
- moved U1 13.3 mm to (7.00, 7.00), flipped to the top, turned to 270 degrees
- moved C9 12.9 mm to (10.4, 7.94)
- moved C13 12.6 mm to (7.50, 1.50)
- moved C4 11.8 mm to (4.44, 12.6), turned to 90 degrees
- moved C7 11.4 mm to (22.9, 1.62), turned to 270 degrees
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- renumbered C23 to C17, TP12 to TP4, TP13 to TP5
Connections:
- net 3.3V: now also C10.1, C6.1, R5.1, U2.6, U3.2, U4.2; no longer C12.1, C13.1, R3.1, U1.2, U2.2, U3.6
- net CLK_EN: now also R1.1; no longer R2.1
- net D0: now also U1.45; no longer U4.45
- net D1: now also U1.46; no longer U4.46
- net D10: now also U1.10; no longer U4.10
- net D11: now also U1.11; no longer U4.11
- net D2: now also U1.47; no longer U4.47
- net D3: now also U1.48; no longer U4.48
- net D4: now also U1.1; no longer U4.1
- net D5: now also U1.2; no longer U4.2
- net D6: now also U1.3; no longer U4.3
- net D7: now also U1.7; no longer U4.7
- net D8: now also U1.8; no longer U4.8
- net D9: now also U1.9; no longer U4.9
- net GND: now also C1.1, C15.2, C16.2, C18.2, C6.2, R4.1, R6.2, U1.25, U1.30, U1.35, U1.39, U1.44, U1.6, U2.2, U2.3, U4.5, U4.7, U4.8, U4.9; no longer C1.2, C20.2, C21.2, C22.2, C6.1, R4.2, R6.1, U1.5, U1.7, U1.8, U1.9, U3.2, U3.3, U4.25, U4.30, U4.35, U4.39, U4.44, U4.6
- net HSYNC: now also U1.29; no longer U4.29
- net N$1: now also R2.1; no longer R1.1
- net N$10: now also U1.26; no longer U4.26
- net N$2: now also R2.2, U1.5; no longer R1.2, U4.5
- net N$3: now also U1.16; no longer U4.16
- net N$4: now also U1.15; no longer U4.15
- net N$5: now also R3.1, R4.2, U1.24; no longer R5.1, R6.2, U4.24
- net N$6: now also U1.17; no longer U4.17
- net N$7: now also U1.23; no longer U4.23
- net N$8: now also U1.27; no longer U4.27
- net N$9: now also U1.22; no longer U4.22
- net PIXCLK: now also U1.13; no longer U4.13
- net VAA: now also C11.1, C12.1, C13.1, TP9.TP, U1.34, U1.36, U1.40, U4.1; no longer C10.1, C22.1, C4.1, TP8.TP, U2.1, U4.34, U4.36, U4.40
- net VAA_PIX: now also C16.1, C7.1, TP10.TP, U1.37, U1.38, U4.3; no longer C11.1, C5.1, TP9.TP, U2.3, U4.37, U4.38
- net VDD: now also C2.1, C3.1, TP6.TP, U1.14, U1.19, U2.1; no longer C1.1, C7.1, TP3.TP, U3.1, U4.14, U4.19
- net VDD_IO: now also C1.2, C18.1, C4.1, C5.1, R1.2, R3.2, TP8.TP, U1.12, U1.18, U3.3; no longer C2.1, C20.1, C6.2, C8.1, R2.2, R5.2, TP2.TP, U1.3, U4.12, U4.18
- net VDD_PLL: now also C15.1, C8.1, TP7.TP, U1.4, U3.1; no longer C21.1, C3.1, TP1.TP, U1.1, U4.4
- net VREG_EN: now also R5.2, R6.1, TP1.TP, TP2.TP, TP3.TP, U3.6, U4.4, U4.6; no longer R3.2, R4.1, TP10.TP, TP11.TP, TP29.TP, U1.4, U1.6, U2.6
- net VSYNC: now also U1.28; no longer U4.28
Other:
- board text added: "OCBv1 == Oresat Camera Board v1"
- board text added: "OCBv1 OLIVER REW"
- board text removed: "AR013X-DEV-BOARD REV.3 ORESAT 2018-12-26 OLIVER REW"
- board text removed: "CUT HERE"
- board text removed: "TEMP SENSOR I2C ADDRS FRONT:0x1B BACK:0x19"
- board text removed: "TODO Enable TPs screw exposed copper ground plane thermals?"
