File: oresat-camera-hardware/oresat-camera-board/AR0130_DEV_BOARD.sch (EAGLE design)
At the start: 41 parts, among them J1 4-1734742-0, U1 TPS71928-28DRVT, U2 TPS71928-28DRVT, U3 TPS70618DRVR, U4 AR0134CSSM00SPCA0, X1 KC2520B27.0000C10E00

Commit message: some final touchs, think it's ready for review
Parts:
- removed C20, C21, C22, C23: 0.1uF, oresat-rcl:C-EU0402-B-NOSILK
- removed TP11, TP29: TPTP06R, J-TestPoint-Small:TPTP06R
- added C15, C18: 2.2uF, oresat-rcl:C-EU0603-C-NOSILK
- added C16: 10uF, oresat-rcl:C-EU0603-C-NOSILK
- added C17: 0.1uF, oresat-rcl:C-EU0402-B-NOSILK
- added TP6, TP7: TPTP06R, J-TestPoint-Small:TPTP06R
- C1: value 10uF -> 10nF; device oresat-rcl:C-EU0603-C-NOSILK -> oresat-rcl:C-EU0402-A-NOSILK
- C10: value 2.2uF -> 1.0uF
- C12: value 1.0uF -> 10uF
- C13: value 1.0uF -> 0.1uF; device oresat-rcl:C-EU0603-C-NOSILK -> oresat-rcl:C-EU0402-B-NOSILK
- C19: value 0.1uF -> 2.2uF; device oresat-rcl:C-EU0402-B-NOSILK -> oresat-rcl:C-EU0603-C-NOSILK
- C3, C5: value 10uF -> 0.1uF; device oresat-rcl:C-EU0603-C-NOSILK -> oresat-rcl:C-EU0402-B-NOSILK
- C6: value 10nF -> 1.0uF; device oresat-rcl:C-EU0402-A-NOSILK -> oresat-rcl:C-EU0603-C-NOSILK
- C8: value 2.2uF -> 10uF
- C9: value 2.2uF -> 0.1uF; device oresat-rcl:C-EU0603-C-NOSILK -> oresat-rcl:C-EU0402-B-NOSILK
- R1: value 100 -> 10k
- R2: value 10k -> 100
- R3: value 10K -> 10k
- R4: value DNP -> 10k
- R5: value 10k -> 10K
- R6: value 10k -> DNP
- U1: value TPS71928-28DRVT -> AR0134CSSM00SPCA0; device U-TI-TPS71928-28-VoltageReg:TPS71928-28DRVT -> U-ONSemi-AR0134:AR0134CSSM00SPCA0
- U2: value TPS71928-28DRVT -> TPS70618DRVR; device U-TI-TPS71928-28-VoltageReg:TPS71928-28DRVT -> U-TI-TPS70618-VoltageReg:TPS70618DRVR
- U3: value TPS70618DRVR -> TPS71928-28DRVT; device U-TI-TPS70618-VoltageReg:TPS70618DRVR -> U-TI-TPS71928-28-VoltageReg:TPS71928-28DRVT
- U4: value AR0134CSSM00SPCA0 -> TPS71928-28DRVT; device U-ONSemi-AR0134:AR0134CSSM00SPCA0 -> U-TI-TPS71928-28-VoltageReg:TPS71928-28DRVT
- renumbered TP12 to TP4, TP13 to TP5
Connections:
- net 3.3V: now also C10.1, C6.1, R5.1, U4.VIN; no longer C12.1, C13.1, R3.1, U1.VIN
- net CLK_EN: now also R1.1; no longer R2.1
- net D0: now also U1.DOUT0; no longer U4.DOUT0
- net D1: now also U1.DOUT1; no longer U4.DOUT1
- net D10: now also U1.DOUT10; no longer U4.DOUT10
- net D11: now also U1.DOUT11; no longer U4.DOUT11
- net D2: now also U1.DOUT2; no longer U4.DOUT2
- net D3: now also U1.DOUT3; no longer U4.DOUT3
- net D4: now also U1.DOUT4; no longer U4.DOUT4
- net D5: now also U1.DOUT5; no longer U4.DOUT5
- net D6: now also U1.DOUT6; no longer U4.DOUT6
- net D7: now also U1.DOUT7; no longer U4.DOUT7
- net D8: now also U1.DOUT8; no longer U4.DOUT8
- net D9: now also U1.DOUT9; no longer U4.DOUT9
- net GND: now also C1.1, C15.2, C16.2, C17.2, C18.2, C6.2, R4.1, R6.2, U1.AGND, U1.DGND, U4.GND; no longer C1.2, C20.2, C21.2, C22.2, C23.2, C6.1, R4.2, R6.1, U1.GND, U4.AGND, U4.DGND
- net HSYNC: now also U1.LINEVALID; no longer U4.LINEVALID
- net N$1: now also R2.1; no longer R1.1
- net N$10: now also U1.FLASH; no longer U4.FLASH
- net N$2: now also R2.2, U1.EXTCLK; no longer R1.2, U4.EXTCLK
- net N$3: now also U1.SDATA; no longer U4.SDATA
- net N$4: now also U1.SCLK; no longer U4.SCLK
- net N$5: now also R3.1, R4.2, U1.SADDR; no longer R5.1, R6.2, U4.SADDR
- net N$6: now also U1.!RESET; no longer U4.!RESET
- net N$7: now also U1.!OE; no longer U4.!OE
- net N$8: now also U1.TRIGGER; no longer U4.TRIGGER
- net N$9: now also U1.STANDBY; no longer U4.STANDBY
- net PIXCLK: now also U1.PIXCLK; no longer U4.PIXCLK
- net VAA: now also C11.1, C12.1, C13.1, TP9.TP, U1.VAA, U4.OUT1; no longer C10.1, C22.1, C4.1, TP8.TP, U2.OUT1, U4.VAA
- net VAA_PIX: now also C16.1, C17.1, C7.1, TP10.TP, U1.VAA_PIX, U4.OUT2; no longer C11.1, C23.1, C5.1, TP9.TP, U2.OUT2, U4.VAA_PIX
- net VDD: now also C2.1, C3.1, TP6.TP, U1.VDD, U2.OUT1; no longer C1.1, C7.1, TP3.TP, U3.OUT1, U4.VDD
- net VDD_IO: now also C1.2, C18.1, C4.1, C5.1, R1.2, R3.2, TP8.TP, U1.VDD_IO, U3.OUT2; no longer C2.1, C20.1, C6.2, C8.1, R2.2, R5.2, TP2.TP, U1.OUT2, U4.VDD_IO
- net VDD_PLL: now also C15.1, C8.1, TP7.TP, U1.VDD_PLL, U3.OUT1; no longer C21.1, C3.1, TP1.TP, U1.OUT1, U4.VDD_PLL
- net VREG_EN: now also R5.2, R6.1, TP1.TP, TP2.TP, TP3.TP, U3.EN2, U4.EN1, U4.EN2; no longer R3.2, R4.1, TP10.TP, TP11.TP, TP29.TP, U1.EN1, U1.EN2, U2.EN2
- net VSYNC: now also U1.FRAME_VALID; no longer U4.FRAME_VALID
Other:
- note added: "36 Pin connector"
- note added: "Image Sensor Caps"
- moved on the sheet: C1, C10, C11, C12, C13, C14, C19, C2, C3, C4, C5, C6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
