File: oresat-camera-hardware/oresat-camera-card-v0/oresat-camera-card-v0.sch (EAGLE design)
At the start: 302 parts, among them J1 J-SAMTEC-TFM-110-X1-XXX-D-RA, J2 U.FL, J3 U.FL, J4 U.FL, J5 DM3BT-DSF-PEJS, J6 J-SAMTEC-TFM-120-X1-XXX-D-RA, J8 3-1734592-64-1734592-0, Q1 DMP2240UDM, Q2 MMBT2907, Q3 MOSFET-PCH-SOT23-6, Q4 MOSFET-PCH-SOT23-6, Q5 PMV45EN, Q6 PMV45EN, U1 OSD3358-512M-BSM, U11 SN74LVC8T245MPWREPPW24-M, U12 TCA9509DGKRDGK8-M, U13 TLVH431, U2 TCAN330, U3 MAX7310ATE, U4 MAX4211CETE, U5 TPS62112, U6 CLVCH16T245MDGGREP, U7 MCP1703A, U8 SN74LVC1G07DCK, U9 TPS2051CDBVR, Y1 ABS07-32.768KHZ-T, Y2 24MHz

Commit message: schematic updates
Parts:
- removed C20: 18pF, 50V, oresat-rcl:C-EU0603-A-NOSILK
- removed CM1, CM2, CM3: J-MOLEX-SMPM-73300-003X, J-Molex-SMPM-73300-003X:J-MOLEX-SMPM-73300-003X
- removed J3, J4: U.FL, SparkFun-Connectors:U.FL2PIN
- removed J9: (no value), SparkFun-Connectors:USB_MICRO-B_FEMALE-SMT
- removed JP9: (no value), pinhead:PINHD-1X10
- removed R41: 1M, 1%, oresat-rcl:R-US_0603-A-NOSILK
- removed Y1: ABS07-32.768KHZ-T, X-Abracon-ABS07-32.768KHZ-T:ABS07-32.768KHZ-T
- added TP123: TEST-POINT, Tova:TEST-POINT
- added TP124, TP125, TP126, TP127, TP128: TEST-POINT3X4, SparkFun-Connectors:TEST-POINT3X4
- C19: value 18pF, 50V -> 100nF
- J1: value J-SAMTEC-TFM-110-X1-XXX-D-RA -> (none); device J-Samtec-TFM-110-X1-XXX-D-RA:J-SAMTEC-TFM-110-X1-XXX-D-RA -> SparkFun-Connectors:USB_MICRO-B_FEMALE-SMT; MFR Samtec -> (none); MPN TFM-110-01-L-D-RA -> (none)
- J2: value U.FL -> (none); device SparkFun-Connectors:U.FL2PIN -> SparkFun-Connectors:CONN_03LONGPADS
Connections:
- removed net AUX_!SHUTDOWN: J1.19, J1.20, JP9.10
- removed net AUX_CAN1_H: J1.13, J1.14, JP9.7
- removed net AUX_CAN1_L: J1.15, J1.16, JP9.8
- removed net AUX_CAN2_H: J1.1, J1.2, JP9.1
- removed net AUX_CAN2_L: J1.3, J1.4, JP9.2
- removed net AUX_GND1: J1.17, J1.18, JP9.9
- removed net AUX_GND2: J1.11, J1.12, JP9.6
- removed net AUX_GND3: J1.10, J1.9, JP9.5
- removed net AUX_VBUS1: J1.7, J1.8, JP9.4
- removed net AUX_VBUS2: J1.5, J1.6, JP9.3
- removed net N$300: CM3.CENTER, J4.SIGNAL
- removed net OSC1_GND: C19.1, C20.1, U1B.OSC1_GND
- removed net OSC1_IN: C20.2, R41.2, U1B.OSC1_IN, Y1.P$2
- removed net OSC1_OUT: C19.2, R41.1, U1B.OSC1_OUT, Y1.P$1
- removed net RF1: CM1.CENTER, J2.SIGNAL
- removed net RF2: CM2.CENTER, J3.SIGNAL
- new net N$80: C19.1, J1.SHIELD
- new net N$81: J7.SHIELD
- net 3.3V: now also D5.A
- net CAN2_H: now also J2.2
- net CAN2_L: now also J2.1
- net GND: now also C19.2, J1.GND, J2.3; no longer CM1.SHIELD, CM1.SHIELD1, CM1.SHIELD2, CM1.SHIELD3, CM2.SHIELD, CM2.SHIELD1, CM2.SHIELD2, CM2.SHIELD3, CM3.SHIELD, CM3.SHIELD1, CM3.SHIELD2, CM3.SHIELD3, J2.GND, J3.GND, J4.GND, J7.SHIELD, J9.GND, J9.SHIELD
- net N$405: no longer D5.A
- net N$525: now also TP123.1
- net N$611: now also J1.D-, TP126.1; no longer J9.D-
- net N$612: now also J1.D+, TP127.1; no longer J9.D+
- net N$613: now also J1.ID, TP128.1; no longer J9.ID
- net N$614: now also J1.VBUS; no longer J9.VBUS
- net N$617: now also TP124.1
- net N$618: now also TP125.1
Other:
- note added: "Camera Control Level Shifter"
- note added: "Camera Output Level Shifter"
- note added: "See Connectors Sheet"
- note added: "TODO Do we really want to remove the PWR button? Should we connect this to the OPD?"
- note added: "TODO GND test points"
- note added: "USB Client Connector"
- note added: "USB Host Connector"
- note removed: "32.768KHz RTC XO"
- note removed: "Auxiliary Connector"
- note removed: "Camera Control Transceiver"
- note removed: "Camera Output Transceiver"
- note removed: "DNP"
- note removed: "RF connections and test points"
- note removed: "TODO MISC GND test points test points for all unconnected pins"
- note removed: "TODO should VTREF be connected to 3.3V"

Commit message: started layout
Parts:
- removed FB3: 30Ω/1.8A, SparkFun-Coils:FERRITE_BEAD-0603
- removed H1, H2, H3, H4: STAND-OFFTIGHT, SparkFun-Hardware:STAND-OFFTIGHT
- removed J7: (no value), SparkFun-Connectors:USB_MICRO-B_FEMALE-SMT
- added J4: (no value), J-Wurth-629105136821-Micro-USB-A:MICRO-USB-SOCKET
- added TP129, TP130, TP131, TP132, TP133: TEST-POINT3X4, SparkFun-Connectors:TEST-POINT3X4
- J1: device SparkFun-Connectors:USB_MICRO-B_FEMALE-SMT -> J-Wurth-629105136821-Micro-USB-A:MICRO-USB-SOCKET
- renumbered RCLAMP0504FB to U16, RCLAMP0504FB1 to U14, U$2 to U15
Connections:
- removed net N$20: J7.ID, TP7.1
- removed net N$611: J1.D-, TP126.1, U16.I1, U1B.USB0_DM
- removed net N$612: J1.D+, TP127.1, U16.I2, U1B.USB0_DP
- removed net N$613: J1.ID, TP128.1, U16.I3, U1B.USB0_ID
- removed net N$614: FB1.1, J1.VBUS
- removed net N$615: FB2.2, J7.VBUS
- removed net N$616: FB3.1, U1B.USB1_VBUS
- removed net N$617: J7.D-, TP124.1, U14.I1, U1B.USB1_DM
- removed net N$618: J7.D+, TP125.1, U14.I2, U1B.USB1_DP
- removed net N$80: C19.1, J1.SHIELD
- removed net N$81: J7.SHIELD
- new net N$82: TP131.1, U1C.GPMC_A9
- new net N$83: TP132.1, U1C.GPMC_A10
- new net N$84: TP133.1, U1C.GPMC_A11
- new net N$85: TP129.1, U1C.GPMC_CSN0
- new net N$86: TP130.1, U1C.GPMC_CSN3
- new net USB_CLI_DM: J4.D-, TP126.1, U16.I3, U1B.USB0_DM
- new net USB_CLI_DP: J4.D+, TP127.1, U16.I2, U1B.USB0_DP
- new net USB_CLI_ID: J4.ID, TP128.1, U16.I1, U1B.USB0_ID
- new net USB_CLI_SHIELD: C19.2, J4.SHIELD
- new net USB_CLI_VBUS: FB1.1, J4.VBUS
- new net USB_HO_DM: J1.D-, TP124.1, U14.I4, U1B.USB1_DM
- new net USB_HO_DP: J1.D+, TP125.1, U14.I1, U1B.USB1_DP
- new net USB_HO_ID: J1.ID, TP7.1
- new net USB_HO_VBUS: FB2.2, J1.VBUS
- net !OE_E: now also J8.26, U11.A5; no longer J8.12, U11.A4
- net !RESET_E: now also J8.24, U11.A3; no longer J8.11, U11.A5
- net 3.3V: now also J8.31, J8.32, J8.33; no longer J8.4, J8.5, J8.6
- net CAM_OE: now also U11.B5; no longer U11.B4
- net CLK_EN: now also U11.B2; no longer U11.B1
- net CLK_EN_E: now also J8.23, U11.A2; no longer J8.16, U11.A1
- net D0_E: now also J8.12, U6.1B7; no longer J8.20, U6.2B7
- net D0_I: now also U6.1A7; no longer U6.2A7
- net D10_E: now also J8.16, U6.1B3; no longer J8.28, U6.1B7
- net D10_I: now also U6.1A3; no longer U6.1A7
- net D11_E: now also J8.17, U6.1B2; no longer J8.27, U6.1B8
- net D11_I: now also U6.1A2; no longer U6.1A8
- net D1_E: now also J8.11, U6.1B8; no longer J8.21, U6.2B6
- net D1_I: now also U6.1A8; no longer U6.2A6
- net D2_E: now also J8.10, U6.2B1; no longer J8.22, U6.2B5
- net D2_I: now also U6.2A1; no longer U6.2A5
- net D3_E: now also J8.9, U6.2B2; no longer J8.23, U6.2B4
- net D3_I: now also U6.2A2; no longer U6.2A4
- net D4_E: now also J8.8; no longer J8.24
- net D5_E: now also J8.7, U6.2B4; no longer J8.25, U6.2B2
- net D5_I: now also U6.2A4; no longer U6.2A2
- net D6_E: now also J8.6, U6.2B5; no longer J8.26, U6.2B1
- net D6_I: now also U6.2A5; no longer U6.2A1
- net D7_E: now also J8.13, U6.1B6; no longer J8.31, U6.1B4
- net D7_I: now also U6.1A6; no longer U6.1A4
- net D8_E: now also J8.14; no longer J8.30
- net D9_E: now also J8.15, U6.1B4; no longer J8.29, U6.1B6
- net D9_I: now also U6.1A4; no longer U6.1A6
- net FLASH: now also U6.1A1; no longer U6.2A8
- net FLASH_E: now also J8.28, U6.1B1; no longer J8.15, U6.2B8
- net GND: now also C19.1, J1.SHIELD, J4.GND, J8.20, J8.34; no longer C19.2, J7.GND, J8.17, J8.3
- net HSYNC_E: now also J8.4, U6.2B7; no longer J8.33, U6.1B2
- net HSYNC_I: now also U6.2A7; no longer U6.1A2
- net I2C2_SCL: now also J8.21, R60.2; no longer J8.10, R59.2
- net I2C2_SDA: now also J8.22, R59.2; no longer J8.9, R60.2
- net N$10: now also R50.66; no longer R50.44
- net N$4: now also R50.99; no longer R50.11
- net N$5: now also R50.22; no longer R50.99
- net N$6: now also R50.88; no longer R50.22
- net N$641: now also R69.66; no longer R69.22
- net N$642: now also R54.11; no longer R69.88
- net N$643: now also R54.99; no longer R69.33
- net N$646: now also R69.33; no longer R69.66
- net N$647: now also R54.88; no longer R54.11
- net N$648: now also R54.22; no longer R54.99
- net N$649: now also R69.22; no longer R69.99
- net N$651: now also R69.88; no longer R69.11
- net N$652: now also R54.33; no longer R54.22
- net N$7: now also R50.33; no longer R50.88
- net N$8: now also R50.77; no longer R50.33
- net N$9: now also R50.44; no longer R50.77
- net PIXCLK_E: now also J8.5, U6.2B6; no longer J8.32, U6.1B3
- net PIXCLK_I: now also U6.2A6; no longer U6.1A3
- net RESET: now also U11.B3; no longer U11.B5
- net SADDR_E: now also J8.27; no longer J8.8
- net STANDBY: now also U11.B4; no longer U11.B2
- net STANDBY_E: now also J8.25, U11.A4; no longer J8.14, U11.A2
- net TRIGGER: now also U11.B7; no longer U11.B3
- net TRIGGER_E: now also J8.29, U11.A7; no longer J8.13, U11.A3
- net VOUT_USB: now also U1B.USB1_VBUS; no longer FB3.2
- net VREG_EN: now also U11.B8; no longer U11.B7
- net VREG_EN_E: now also J8.30, U11.A8; no longer J8.7, U11.A7
- net VSYNC_E: now also J8.3, U6.2B8; no longer J8.34, U6.1B1
- net VSYNC_I: now also U6.2A8; no longer U6.1A1
Other:
- moved on the sheet: C43, C44, R50, R54, R59, R60, R63, R69, TP106, TP107, TP124, TP125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

Commit message: saved my octavo card work so I don't cry if it gets lost some how
Parts:
- removed C16, C34: 22uF, oresat-rcl:C-EUC1210
- removed J2: (no value), SparkFun-Connectors:CONN_03LONGPADS
- removed JP10: (no value), pinhead:PINHD-2X5
- removed JP11: (no value), pinhead:PINHD-2X6
- removed S1: MOMENTARY-SWITCH-SPST-SMD-4.6X2.8MM, SparkFun-Switches:MOMENTARY-SWITCH-SPST-SMD-4.6X2.8MM
- added J3: (no value), SparkFun-Connectors:CONN_02PTH3
- added JP5, JP6: JUMPER-SMT_2_NC_TRACE_SILK, SparkFun-Jumpers:JUMPER-SMT_2_NC_TRACE_SILK
- added TP134, TP135, TP136, TP137, TP138, TP139, TP140, TP141: TEST-POINT3X4, SparkFun-Connectors:TEST-POINT3X4
- Q2: device OSD3358-SM-RED Platform:MMBT2907SMD -> Q-Diodesinc-MMBT2907-PNP:MMBT2907SMD
- TP123: value TEST-POINT -> TEST-POINT3X4; device Tova:TEST-POINT -> SparkFun-Connectors:TEST-POINT3X4
- U13: device OSD3358-SM-RED Platform:TLVH431 -> U-TI-TLVH431-Shunt-Regulator:TLVH431
- U8: device GHI-IC:SN74LVC1G07DCK -> U-TI-SN74LVC1G07DCK-Buffer:SN74LVC1G07DCK
- renumbered R54 to R41
Connections:
- net USB_CLI_DM renamed USB_CLI_N
- net USB_CLI_DP renamed USB_CLI_P
- net USB_HO_DM renamed USB_HO_N
- net USB_HO_DP renamed USB_HO_P
- removed net N$528: D5.C, R39.1
- removed net N$605: D6.C, R42.1
- removed net N$606: D7.C, R43.1
- removed net N$607: D8.C, R44.1
- removed net N$608: D9.C, R45.1
- new net N$20: JP5.2, Q2.E, R66.2, R68.2
- new net N$80: D8.A, R44.2
- new net N$81: D7.A, R43.2
- new net N$87: D6.A, R42.2
- new net N$88: D5.A, R39.2
- new net N$89: TP135.1, U1B.OSC1_IN
- new net N$90: TP134.1, U1B.OSC1_OUT
- new net N$91: TP26.1, U1B.OSC1_GND
- new net N$92: TP136.1, U1B.USB1_CE
- new net N$93: TP140.1, U1C.GPMC_ADVN_ALE
- new net N$94: TP139.1, U1C.GPMC_BEN0_CLE
- new net N$95: TP138.1, U1C.GPMC_WEN
- new net N$96: TP137.1, U1C.GPMC_OEN_REN
- new net N$97: TP141.1, U1D.MII1_TX_EN
- net !SHUTDOWN: no longer JP10.10, JP10.9
- net 3.3V: now also R39.1, R56.2; no longer D5.A, TP26.1
- net 5V_IN: no longer C16.1
- net CAN1_H: no longer JP10.5, JP10.6
- net CAN1_L: no longer JP10.7, JP10.8
- net CAN2_H: no longer J2.2, JP11.11
- net CAN2_L: no longer J2.1, JP11.12
- net GND: now also D5.C, D6.C, D7.C, D8.C, D9.C, J3.1; no longer C16.2, C34.2, J2.3, JP11.10, JP11.9, R39.2, R42.2, R43.2, R44.2, R45.2, S1.1
- net N$10: now also TP39.1, U1C.SPI0_CS1
- net N$2: now also D9.A, R45.2; no longer R56.2, TP43.1
- net N$26: now also JP5.1; no longer Q2.E, R66.2, R68.2
- net N$32: now also JP6.1, TP28.1, U1A.SYS_RTC_1P8V@1, U1A.SYS_RTC_1P8V@2; no longer TP39.1, U1C.SPI0_CS1
- net N$407: now also JP6.2; no longer TP28.1, U1A.SYS_RTC_1P8V@1, U1A.SYS_RTC_1P8V@2
- net N$525: now also J3.2; no longer S1.2, TP123.1
- net N$585: now also R53.88; no longer R53.44
- net N$587: now also R52.11; no longer R52.99
- net N$588: now also R52.99; no longer R52.22
- net N$601: now also R51.44; no longer R51.22
- net N$629: now also R52.22; no longer R52.11
- net N$630: now also R53.11; no longer R53.77
- net N$631: now also R53.99; no longer R53.33
- net N$632: now also R53.22; no longer R53.88
- net N$633: now also R53.44; no longer R53.22
- net N$634: now also R53.77; no longer R53.99
- net N$635: now also R51.11; no longer R51.66
- net N$636: now also R51.99; no longer R51.44
- net N$637: now also R51.88; no longer R51.77
- net N$638: now also R51.77; no longer R51.33
- net N$639: now also R51.66; no longer R51.88
- net N$653: now also R42.1; no longer D6.A
- net N$654: now also R43.1; no longer D7.A
- net N$655: now also R44.1; no longer D8.A
- net N$656: now also R45.1; no longer D9.A
- net PMIC_MUX_IN: now also TP43.1
- net SPARE1: no longer JP11.8
- net SPARE2: no longer JP11.7
- net SPARE3: no longer JP11.6
- net SPARE4: no longer JP11.5
- net SPARE5: no longer JP11.4
- net SPARE6: no longer JP11.3
- net SPARE7: no longer JP11.2
- net VBUS: no longer JP10.1, JP10.2, JP10.3, JP10.4
- net VIN_USB: no longer C34.1
- net VOUT_USB: now also TP123.1
Other:
- note added: "Power Button TODO Label in silk TODO does OPD need this?"
- note added: "TODO add optional resistors from AM335X datasheet"
- note added: "VSS_OSC"
- note added: "XTALIN"
- note added: "XTALOUT"
- note removed: "POWER BUTTON"
- note removed: "TODO Do we really want to remove the PWR button? Should we connect this to the OPD?"
- moved on the sheet: D5, Q2, R39, R42, R43, R44, R45, R66, R67, R68, TP39, TP43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

Commit message: more cleanup
Parts:
- removed C19: 100nF, oresat-rcl:C-EU0603-A-NOSILK
- removed J1, J4: (no value), J-Wurth-629105136821-Micro-USB-A:MICRO-USB-SOCKET
- added J2: 2-1734592-0, J-TEConnectivity-X-1734592-X:2-1734592-0
- J8: device J-TEConnectivity-3-1734592-6:3-1734592-64-1734592-0 -> J-TEConnectivity-X-1734592-X:3-1734592-64-1734592-0
Connections:
- removed net USB_CLI_SHIELD: C19.2, J4.SHIELD
- net GND: now also J2.1, J2.10, J2.11, J2.13, J2.16, J2.19, J2.2, J2.20, J2.4, J2.7, J2.PAD; no longer C19.1, J1.GND, J1.SHIELD, J4.GND
- net USB_CLI_ID: now also J2.12; no longer J4.ID
- net USB_CLI_N: now also J2.15; no longer J4.D-
- net USB_CLI_P: now also J2.14; no longer J4.D+
- net USB_CLI_VBUS: now also J2.17, J2.18; no longer J4.VBUS
- net USB_HO_ID: now also J2.3; no longer J1.ID
- net USB_HO_N: now also J2.6; no longer J1.D-
- net USB_HO_P: now also J2.5; no longer J1.D+
- net USB_HO_VBUS: now also J2.8, J2.9; no longer J1.VBUS
Other:
- note added: "TODO cap between client shield and ground on breakout board"
- note added: "USB Client"
- note added: "USB Host"
- note removed: "USB Client Connector"
- note removed: "USB Host Connector"

Commit message: made USB breakout board, added OPD schematic
Parts:
- removed C8: TBD, rcl_custom:C-EU0402-B-NOSILK
- removed U7: MCP1703A, v-reg:XC63FPM
- added Q7: DMP2240UDM, Q-MOSFET-PCH-dual-SOT23-6:MOSFET-PCH-SOT23-6
- added R54, R72, R73: NP, rcl_custom:R-US_0402-B-NOSILK
- added R70: 100, rcl_custom:R-US_0402-B-NOSILK
- added R71: 10k, rcl_custom:R-US_0402-B-NOSILK
- added TP142: TEST-POINT, Tova:TEST-POINT
- added U$2, U$4: MIC842, Q-Microchip-MIC842-Comparator:MIC842
- C10, C5: device oresat-rcl:C-EU0603-B-NOSILK -> oresat-rcl:C-EU0603-A-NOSILK
- C2: device rcl_custom:C-EU0402-B-NOSILK -> oresat-rcl:C-EU0603-A-NOSILK
- C4: value 1u -> NP; device oresat-rcl:C-EU0603-B-NOSILK -> oresat-rcl:C-EU0805-B-NOSILK; DIS Digi-Key -> (none); DPN 1276-1001-1-ND -> (none); MFR Samsung -> (none); MPN CL05B104KO5NNNC -> (none)
- C6: value TBD -> NP; device rcl_custom:C-EU0402-B-NOSILK -> oresat-rcl:C-EU0805-B-NOSILK; DIS Digi-Key -> (none); DPN 1276-1001-1-ND -> (none); MFR Samsung -> (none); MPN CL05B104KO5NNNC -> (none)
- R10, R27, R28, R30, R31, R32, R33, R34, R35, R36, R37, R38, R7: device rcl_custom:R-US_0402-B-NOSILK -> oresat-rcl:R-US_0603-A-NOSILK
- R16, R18: value 10k -> 47k
- R24: value 100 -> NP
- TP7: value TEST-POINT3X4 -> TEST-POINT; device SparkFun-Connectors:TEST-POINT3X4 -> Tova:TEST-POINT
Connections:
- net !SHUTDOWN renamed !SD
- net N$598 renamed IOUT
- net N$600 renamed POUT
- removed net N$398: C4.1, Q3.S, R29.2, R35.2, U4.RS-, U7.IN
- removed net N$482: TP3.1, U3.IO4
- removed net N$518: TP4.1, U3.IO5
- removed net N$523: TP5.1, U3.IO6
- removed net N$573: R12.2, TP10.1, U3.IO7
- removed net N$581: C8.2, Q1.2.G, R16.2, R18.1
- removed net SPARE6: J6.3, J6.4
- removed net SPARE7: J6.1, J6.2
- removed net USB_HO_ID: J2.3, TP7.1
- new net BOOT0: U3.IO5
- new net N$385: R16.1, R18.1, TP5.1, U3.IO6
- new net N$479: Q7.1.S, R70.2
- new net N$99: Q3.S, R29.2, R35.2, U4.RS-
- new net PB6/SCL: R18.2, U3.IO0
- new net PB7/SDA: R16.2, U3.IO1
- net CAN2_H: now also J6.17, J6.18; no longer J6.21, J6.22
- net CAN2_L: now also J6.19, J6.20; no longer J6.23, J6.24
- net CB-RESET: now also U3.IO4, U4.CIN2-; no longer U3.IO1, U4.CIN2+
- net CB_CTRL: now also TP3.1
- net GND: now also C6.2, J2.3, J6.27, J6.28, R71.1, U$2.GND, U$4.GND; no longer U7.GND
- net MAX4211-3V3: now also TP10.1, U3.IO7; no longer U7.OUT
- net N$480: now also Q7.1.G, R71.2, TP142.1, U$4.COUT; no longer TP2.1, U3.IO3
- net N$579: no longer C6.1
- net N$580: now also TP7.1, U$2.COUT; no longer C6.2, Q1.2.D
- net N$599: now also U4.CIN2+; no longer U4.CIN2-
- net ON/!OFF: now also R12.2, U3.IO3; no longer U3.IO0
- net OPD_PWR: now also J6.15, J6.16; no longer J6.19, J6.20
- net OPD_SCL: now also J6.13, J6.14, R70.1; no longer J6.17, J6.18, R24.1
- net OPD_SDA: now also J6.11, J6.12; no longer J6.15, J6.16
- net PEN-SCL-FILT: now also C6.1, Q7.1.D, R72.1, R72.2, R73.1, TP2.1, U$4.CIN; no longer R24.2
- net PEN-SDA-FILT: now also C4.1, R24.1, R24.2, R54.1, TP4.1, U$2.CIN; no longer R16.1
- net SPARE1: now also J6.10, J6.9; no longer J6.13, J6.14
- net SPARE2: now also J6.7, J6.8; no longer J6.11, J6.12
- net SPARE3: now also J6.5, J6.6; no longer J6.10, J6.9
- net SPARE4: now also J6.3, J6.4; no longer J6.7, J6.8
- net SPARE5: now also J6.1, J6.2; no longer J6.5, J6.6
- net VBUS: now also J6.21, J6.22, J6.23, J6.24; no longer J6.27, J6.28
- net VPD: now also R54.2, R73.2, U$2.VCC, U$4.VCC; no longer C8.1, Q1.2.S, R18.2
Other:
- note added: "47k forces slow I2C"
- note added: "Place only if I2C pullups not placed."
- moved on the sheet: C1, C2, C4, C5, C6, D1, D4, Q1.1, Q3, Q4, Q5, Q6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
