File: oresat-camera-hardware/star-tracker-camera-board/star-tracker-camera-board.brd (EAGLE design)
At the start: 31.5 x 14 mm, 43 parts, among them J1 4-1734742-0, U1 AR0134CSSM00SPCA0, U2 TPS70618DRVR, U3 TPS71928-28DRVT, U4 TPS71928-28DRVT, X1 KC2520B27.0000C10E00

Commit message: implemented design review changes. Cleaned up the repo a bit. Added generic SPI EEPROM footprint for booting
Parts:
- removed R1: 10k, oresat-rcl:.0402-B
- added R10, R11, R12, R9: 10k, oresat-rcl:.0402-B
- J1: value 4-1734742-0 -> 3-1734742-6; device J-TEConnectivity-4-1734742-0:TE_4-1734742-0 -> J-TEConnectivity-3-1734742-6 :TE_3-1734742-6
- R3, R4, R6, R7, R8: device oresat-rcl:.0402-B -> oresat-rcl:.0402-B-NOSILK
- R5: value 10K -> 10k; device oresat-rcl:.0402-B -> oresat-rcl:.0402-B-NOSILK
- moved TP4 19.6 mm to (15.1, 13.3)
- moved R4 19.3 mm to (21.5, 6.50)
- moved R3 18.1 mm to (20.5, 6.50), turned to 90 degrees
- moved TP8 15.0 mm to (19.5, 8.50)
- moved TP5 14.2 mm to (21.1, 13.3)
- moved TP2 12.6 mm to (24.9, 13.3)
- moved TP1 12.1 mm to (30.4, 13.3)
- moved TP3 11.2 mm to (26.6, 13.3)
- moved C11 10.7 mm to (30.6, 11.4), turned to 90 degrees
- moved C14 10.6 mm to (19.2, 12.4), turned to 270 degrees
- moved C15 10.4 mm to (25.1, 11.4), turned to 90 degrees
- moved C7 10.4 mm to (26.4, 11.4), turned to 90 degrees
- moved U2 10.3 mm to (17.0, 12.0), turned to 90 degrees
- moved C18 10.1 mm to (20.9, 11.4), turned to 90 degrees
- moved C4 9.52 mm to (13.7, 10.3), turned to 180 degrees
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Connections:
- removed net N$10: J1.15, U1.26
- removed net N$3: J1.9, R8.1, U1.16
- removed net N$4: J1.10, R7.1, U1.15
- removed net N$5: J1.8, R3.1, R4.2, U1.24
- removed net N$6: J1.11, U1.17
- removed net N$7: J1.12, U1.23
- removed net N$8: J1.13, U1.27
- removed net N$9: J1.14, U1.22
- new net !OE: J1.11, R11.1, U1.23
- new net !RESET: J1.13, R9.2, U1.17
- new net FLASH: J1.9, U1.26
- new net SADDR: J1.10, R3.1, R4.2, U1.24
- new net SCLK: J1.16, R7.1, U1.15
- new net SDATA: J1.15, R8.1, U1.16
- new net STANDBY: J1.12, R10.1, U1.22
- new net TRIGGER: J1.8, U1.27
- net CLK_EN: now also J1.14, R12.2; no longer J1.16, R1.1
- net D0: now also J1.25; no longer J1.20
- net D1: now also J1.26; no longer J1.21
- net D10: now also J1.21; no longer J1.28
- net D11: now also J1.20; no longer J1.27
- net D2: now also J1.27; no longer J1.22
- net D3: now also J1.28; no longer J1.23
- net D4: now also J1.29; no longer J1.24
- net D5: now also J1.30; no longer J1.25
- net D6: now also J1.31; no longer J1.26
- net D7: now also J1.24; no longer J1.31
- net D8: now also J1.23; no longer J1.30
- net D9: now also J1.22; no longer J1.29
- net GND: now also R12.1, R9.1
- net HSYNC: now also J1.34; no longer J1.33
- net VDD_IO: now also R10.2, R11.2; no longer R1.2
- net VSYNC: now also J1.33; no longer J1.34
Routing:
- net VREG_EN: track 101.6 -> 58.4 mm, vias 12 -> 7
- net N$5: track 32.6 -> 0.00 mm, vias 2 -> 0
- net N$7: track 28.6 -> 0.00 mm, vias 3 -> 0
- net SADDR: track 0.00 -> 28.3 mm, vias 0 -> 1
- net N$4: track 27.6 -> 0.00 mm, vias 2 -> 0
- net TRIGGER: track 0.00 -> 27.4 mm, vias 0 -> 1
- net STANDBY: track 0.00 -> 27.2 mm, vias 0 -> 3
- net N$3: track 27.1 -> 0.00 mm, vias 2 -> 1
- net N$8: track 26.4 -> 0.00 mm, vias 3 -> 0
- net FLASH: track 0.00 -> 25.9 mm, vias 0 -> 1
- net N$10: track 25.6 -> 0.00 mm, vias 3 -> 0
- net N$6: track 25.2 -> 0.00 mm, vias 2 -> 0
- net !OE: track 0.00 -> 25.1 mm, vias 0 -> 2
- net !RESET: track 0.00 -> 25.0 mm, vias 0 -> 2
- net N$9: track 24.6 -> 0.00 mm, vias 2 -> 0
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- added copper zone on layer 1, net VAA
- added copper zone on layer 1, net VDD_IO
- added copper zone on layer 1, net VDD_PLL
Other:
- board text added: "MAKE SURE FFC CONNECTOR IS CORRECT ORIENTATION! CONTACTS MUST BE ON TOP OF CONNECTOR TO MATE WITH OCTAVO CARD. MEASURE TWICE CUT ONCE!!!!"
- board text added: "OCBv2 == Oresat Camera Board v2"
- board text added: "OCBv3 OLIVER REW 2020.05.31"
- board text removed: "OCBv1 == Oresat Camera Board v1"
- board text removed: "OCBv1 OLIVER REW"
