File: hardware/star-tracker-card/star-tracker-card_1.kicad_sch (KiCad schematic)
At the start: 11 parts, among them J1 ORESAT-DEBUG-CONNECTOR-CARD, J4 TFM-120-01-L-D-RA

Commit message: More EAGLE import cleanup
Fixed sheets, did some ERC cleanup, imported into layout, impmorted 4 layer DRC rules.
Parts:
- removed U$1: FLIGHMARKERNEW, star-tracker-card:FLIGHTMARKER_NEW_BOARDS, symbol star-tracker-card-eagle-import:FLIGHMARKERNEW
Other:
- note removed: "1.2"
- note removed: "OreSat Star Tracker: Connectors"
- company: (none) -> Portland State Aerospace Society
- title: (none) -> OreSat Star Tracker
Changed lines of the file:
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@@
 	(generator "eeschema")
 	(generator_version "9.0")
-	(paper "User" 469.9 317.627)
+	(paper "B")
+	(title_block
+		(title "OreSat Star Tracker")
+		(date "2026-01-30")
+		(rev "1.3")
+		(company "Portland State Aerospace Society")
+	)
 	(text "OreSat Power Domain signals\n(See power sheet)"
 		(exclude_from_sim no)
@@
 		)
 	)
-	(text "1.2"
-		(exclude_from_sim no)
-		(at 434.34 290.83 0)
-		(effects
-			(font
-				(size 3.81 3.2385)
-			)
-			(justify left bottom)
-		)
-	)
 	(text "All resistors 0402 +/- 1% unless marked"
 		(exclude_from_sim no)
-		(at 29.21 292.1 0)
+		(at 116.84 261.62 0)
 		(effects
 			(font
@@
 	(text "All caps are 0402 ceramic 10% X5R Vw>=16V unless marked"
 		(exclude_from_sim no)
-		(at 29.21 294.64 0)
+		(at 116.84 264.16 0)
 		(effects
 			(font
@@
 			(font
 				(size 2.54 2.159)
-			)
-			(justify left bottom)
-		)
-	)
-	(text "OreSat Star Tracker: Connectors"
-		(exclude_from_sim no)
-		(at 354.33 270.51 0)
-		(effects
-			(font
-				(size 3.81 3.2385)
 			)
 			(justify left bottom)
@@
 					(reference "J1")
 					(unit 1)
-				)
-			)
-		)
-	)
-	(symbol
-		(lib_id "star-tracker-card-eagle-import:FRAME_B_L")
-		(at 342.9 297.18 0)
-		(unit 2)
-		(exclude_from_sim no)
-		(in_bom yes)
-		(on_board yes)
-		(dnp no)
-		(property "Reference" "#FRAME1"
-			(at 342.9 297.18 0)
-			(effects
-				(font
-					(size 1.27 1.27)
-				)
-				(hide yes)
-			)
-		)
-		(property "Value" "FRAME_B_L"
-			(at 342.9 297.18 0)
-			(effects
-				(font
-					(size 1.27 1.27)
-				)
-				(hide yes)
-			)
-		)
-		(property "Footprint" ""
-			(at 342.9 297.18 0)
-			(effects
-				(font
-					(size 1.27 1.27)
-				)
-				(hide yes)
-			)
-		)
-		(property "Datasheet" ""
-			(at 342.9 297.18 0)
-			(effects
-				(font
-					(size 1.27 1.27)
-				)
-				(hide yes)
-			)
-		)
-		(property "Description" ""
-			(at 342.9 297.18 0)
-			(effects
-				(font
-					(size 1.27 1.27)
-				)
-				(hide yes)
-			)
-		)
-		(instances
-			(project ""
-				(path "/324e9eb5-7420-4b7e-862c-cc20bb28618a/5c15621b-beb3-4a89-9b40-ee1802c4f8e5"
-					(reference "#FRAME1")
-					(unit 2)
 				)
 			)
@@
 	)
 	(symbol
-		(lib_id "star-tracker-card-eagle-import:FLIGHMARKERNEW")
-		(at 264.16 294.64 0)
-		(unit 1)
-		(exclude_from_sim no)
-		(in_bom yes)
-		(on_board yes)
-		(dnp no)
-		(property "Reference" "U$1"
-			(at 264.16 294.64 0)
-			(effects
-				(font
-					(size 1.27 1.27)
-				)
-				(hide yes)
-			)
-		)
-		(property "Value" "FLIGHMARKERNEW"
-			(at 264.16 294.64 0)
-			(effects
-				(font
-					(size 1.27 1.27)
-				)
-				(hide yes)
-			)
-		)
-		(property "Footprint" "star-tracker-card:FLIGHTMARKER_NEW_BOARDS"
-			(at 264.16 294.64 0)
-			(effects
-				(font
-					(size 1.27 1.27)
-				)
-				(hide yes)
-			)
-		)
-		(property "Datasheet" ""
-			(at 264.16 294.64 0)
-			(effects
-				(font
-					(size 1.27 1.27)
-				)
-				(hide yes)
-			)
-		)
-		(property "Description" ""
-			(at 264.16 294.64 0)
-			(effects
-				(font
-					(size 1.27 1.27)
-				)
-				(hide yes)
-			)
-		)
-		(instances
-			(project ""
-				(path "/324e9eb5-7420-4b7e-862c-cc20bb28618a/5c15621b-beb3-4a89-9b40-ee1802c4f8e5"
-					(reference "U$1")
-					(unit 1)
-				)
-			)
-		)
-	)
-	(symbol
-		(lib_id "star-tracker-card-eagle-import:FRAME_B_L")
-		(at 17.78 297.18 0)
-		(unit 1)
-		(exclude_from_sim no)
-		(in_bom yes)
-		(on_board yes)
-		(dnp no)
-		(property "Reference" "#FRAME1"
-			(at 17.78 297.18 0)
-			(effects
-				(font
-					(size 1.27 1.27)
-				)
-				(hide yes)
-			)
-		)
-		(property "Value" "FRAME_B_L"
-			(at 17.78 297.18 0)
-			(effects
-				(font
-					(size 1.27 1.27)
-				)
-				(hide yes)
-			)
-		)
-		(property "Footprint" ""
-			(at 17.78 297.18 0)
-			(effects
-				(font
-					(size 1.27 1.27)
-				)
-				(hide yes)
-			)
-		)
-		(property "Datasheet" ""
-			(at 17.78 297.18 0)
-			(effects
-				(font
-					(size 1.27 1.27)
-				)
-				(hide yes)
-			)
-		)
-		(property "Description" ""
-			(at 17.78 297.18 0)
-			(effects
-				(font
-					(size 1.27 1.27)
-				)
-				(hide yes)
-			)
-		)
-		(instances
-			(project ""
-				(path "/324e9eb5-7420-4b7e-862c-cc20bb28618a/5c15621b-beb3-4a89-9b40-ee1802c4f8e5"
-					(reference "#FRAME1")
-					(unit 1)
-				)
-			)
-		)
-	)
-	(symbol
 		(lib_id "star-tracker-card-eagle-import:ORESAT-CARD-V1.3-STAR-TRACKER")
-		(at 152.4 292.1 0)
+		(at 227.33 256.54 0)
 		(unit 1)
 		(exclude_from_sim no)
@@
 		(dnp no)
 		(property "Reference" "PCB1"
-			(at 152.4 292.1 0)
+			(at 227.33 256.54 0)
 			(effects
 				(font
@@
 		)
 		(property "Value" "ORESAT-CARD-V1.3-STAR-TRACKER"
-			(at 152.4 292.1 0)
+			(at 227.33 256.54 0)
 			(effects
 				(font
@@
 		)
 		(property "Footprint" "star-tracker-card:ORESAT-CARD-V1.3-STAR-TRACKER"
-			(at 152.4 292.1 0)
+			(at 227.33 256.54 0)
 			(effects
 				(font
@@
 		)
 		(property "Datasheet" ""
-			(at 152.4 292.1 0)
+			(at 227.33 256.54 0)
 			(effects
 				(font
@@
 		)
 		(property "Description" ""
-			(at 152.4 292.1 0)
-			(effects
-				(font
+			(at 227.33 256.54 0)
+			(effects
+				(font
