File: hardware/star-tracker-card/star-tracker-card.kicad_pcb (KiCad board)
At the start: 4 copper layers, 99.8 x 94.6 mm, 294 parts, among them J1 ORESAT-DEBUG-CONNECTOR-CARD, J100 DM3BT-DSF-PEJS, J101 3-1734592-64-1734592-0, J3 CONN_03LONGPADS, J4 TFM-120-01-L-D-RA, Q1 MMBT2907, Q2 PMV45EN, Q3 DMP2240UDM, Q4 PMV45EN, Q5 DMP3050LVT-7, Q6 DMP3050LVT-7, U1 RCLAMP0504FB, U10 TLVH431, U11 TCAN330, U12 MIC842LYC5, U13 MIC842LYC5, U14 MAX4211FETE, U15 TPS62112, U16 MAX7310ATE, U17 25AAXX, U2 TS5A21366DCUR, U3 THGBMJG7C2LBAU8, U4 SN74LVC1G07DCK, U5 SN74LVC8T245MPWREPPW24-M, U6 CLVCH16T245MDGGREP, U7 OSD3358-512M-BSM, U8 TLV70028QDDCRQ1, U9 TCA9509DGKRDGK8-M, Y1 24MHz, Y2 ABS07-32.768KHZ-T

Commit message: No ERCs now
Parts:
- removed J3: CONN_03LONGPADS, star-tracker-card:1X03_LONGPADS
- removed JP101, JP104: JUMPER-SMT_2_NC_TRACE_SILK, star-tracker-card:SMT-JUMPER_2_NC_TRACE_SILK
- removed JP102, JP103, JP105, JP106, JP108, JP109, JP110, JP111: JUMPER-SMT_3_1-NC_TRACE_SILK, star-tracker-card:SMT-JUMPER_3_1-NC_TRACE_SILK
- removed JP107: JUMPER-SMT_3_NO_SILK, star-tracker-card:SMT-JUMPER_3_NO_SILK
- removed TP14, TP154, TP156, TP160, TP166, TP60, TP61, TP62, TP71, TP72, TP73: TEST-POINT3X4, oresat-misc:TestPoint_Pad_D1.0mm
- added C47: 100n, oresat-passives:0603-C-NOSILK, F.Cu at (82.7, 116.0)
- added C65: 100n, oresat-passives:0603-C-NOSILK, F.Cu at (82.7, 118.2)
- added C93: 22u, Capacitor_SMD:C_1210_3225Metric, F.Cu at (87.1, 117.1)
- added J6: Conn_01x02, Connector_PinHeader_2.54mm:PinHeader_1x02_P2.54mm_Vertical, F.Cu at (83.0, 103.5)
- added J7: GRPB041VWVN-RC, Connector_PinHeader_1.27mm:PinHeader_1x04_P1.27mm_Vertical, F.Cu at (89.7, 88.6)
- added R78: 10k, oresat-passives:0603-C-NOSILK, F.Cu at (82.7, 120.2)
- Y1: value 24MHz -> ECS-240-12-30BQ-AEN-TR; footprint star-tracker-card:5X3.2-4SMD -> oresat-passives:CRYSTAL-5X3.2-4SMD
- Y2: footprint star-tracker-card:CRYSTAL_3.2X1.5 -> oresat-passives:CRYSTAL_3.2X1.5
- moved TP109 47.6 mm to (82.5, 154.6)
- moved TP183 47.6 mm to (82.5, 161.2)
- moved TP184 47.6 mm to (82.5, 163.5)
- moved TP32 47.6 mm to (82.5, 158.9)
- moved R75 36.4 mm to (87.8, 132.9)
- moved R77 36.4 mm to (87.8, 135.4)
- moved C41 36.4 mm to (87.6, 128.5)
- moved C44 36.4 mm to (87.6, 130.6)
- moved C7 36.4 mm to (87.6, 126.4)
- moved R74 36.4 mm to (83.1, 130.0)
Connections:
- net /SIP A, E ,F/PMIC_PGOOD renamed /SIP A/PMIC_PGOOD
- net Net-(U7A-I2C0_SCL) renamed /SIP A/PMIC_SCL
- net Net-(U7A-I2C0_SDA) renamed /SIP A/PMIC_SDA
- C13 pad 1: /SIP A, E ,F/VIN_USB -> /V_USB
- C18 pad 1: 3.3VA -> Net-(Q1-C)
- C4 pad 1: /SIP A, E ,F/VIN_USB -> Net-(U1-VCC)
- FB2 pad 2: /SIP A, E ,F/VIN_USB -> Net-(U1-VCC)
- J100 pad 1: Net-(J100-DAT2) -> /Camera Logical Level Shifters/D1_I
- J100 pad 2: Net-(J100-DAT3/CS) -> /Camera Logical Level Shifters/D0_I
- J100 pad 7: Net-(J100-DAT0/DO) -> /Camera Logical Level Shifters/D3_I
- J100 pad 8: Net-(J100-DAT1) -> /Camera Logical Level Shifters/D2_I
- J4 pad 1: Net-(J4-Pad1) -> unconnected-(J4-Pad1)
- J4 pad 2: Net-(J4-Pad1) -> unconnected-(J4-Pad2)
- J4 pad 3: Net-(J4-Pad3) -> unconnected-(J4-Pad3)
- J4 pad 4: Net-(J4-Pad3) -> unconnected-(J4-Pad4)
- J4 pad 5: Net-(J4-Pad5) -> unconnected-(J4-Pad5)
- J4 pad 6: Net-(J4-Pad5) -> unconnected-(J4-Pad6)
- Q1 pad B: Net-(U10-CATHODE) -> (no net)
- Q1 pad C: Net-(U10-ANODE) -> (no net)
- Q1 pad E: Net-(JP101-Pad2) -> (no net)
- R23 pad 1: Net-(U10-CATHODE) -> Net-(Q1-B)
- R23 pad 2: Net-(JP101-Pad2) -> Net-(Q1-E)
- R24 pad 2: Net-(R24-22) -> unconnected-(R24-22-Pad2)
- R24 pad 8: Net-(R24-88) -> Net-(J6-Pin_1)
- R24 pad 9: Net-(R24-99) -> unconnected-(R24-99-Pad9)
- R25 pad 3: Net-(R25-33) -> unconnected-(R25-33-Pad3)
- R25 pad 6: Net-(R25-66) -> unconnected-(R25-66-Pad6)
- R25 pad 9: Net-(R25-99) -> unconnected-(R25-99-Pad9)
- R28 pad 2: Net-(JP101-Pad2) -> Net-(Q1-E)
- R31 pad 1: Net-(U10-ANODE) -> Net-(Q1-C)
- R8 pad 2: Net-(J100-DAT3/CS) -> /Camera Logical Level Shifters/D0_I
- R8 pad 4: Net-(J100-DAT1) -> /Camera Logical Level Shifters/D2_I
- R8 pad 7: Net-(J100-DAT0/DO) -> /Camera Logical Level Shifters/D3_I
- R8 pad 9: Net-(J100-DAT2) -> /Camera Logical Level Shifters/D1_I
- TP109 pad 1: Net-(U4-Y) -> /SIP A/nRESET
- TP164 pad 1: 3.3VA -> Net-(Q1-C)
- TP23 pad 1: /SIP C/D3_I -> /Camera Logical Level Shifters/D3_I
- U1 pad 4: unconnected-(U1-I3-Pad4) -> /SIP A/nRESET
- U1 pad 5: /SIP A, E ,F/VIN_USB -> Net-(U1-VCC)
- U10 pad 2: Net-(U10-CATHODE) -> Net-(Q1-B)
- U10 pad 3: Net-(U10-ANODE) -> Net-(Q1-C)
- U2 pad 2: /UART0_TX -> Net-(U16-IO7)
- U2 pad 3: Net-(U16-IO7) -> /UART0_RX
- U2 pad 6: /UART0_RX -> /UART0_TX
- U4 pad 4: Net-(U4-Y) -> /SIP A/nRESET
- U4 pad 5: 3.3VA -> Net-(Q1-C)
- U6 pad 35: /SIP C/D3_I -> /Camera Logical Level Shifters/D3_I
- U7 pad A15: Net-(U7C-MMC0_DAT1) -> /Camera Logical Level Shifters/D2_I
- U7 pad A16: Net-(U7C-MMC0_DAT0) -> /Camera Logical Level Shifters/D3_I
- U7 pad C15: Net-(U7C-MMC0_DAT3) -> /Camera Logical Level Shifters/D0_I
- U7 pad C16: Net-(U7C-MMC0_DAT2) -> /Camera Logical Level Shifters/D1_I
- U7 pad F13: Net-(U7F-VDD_MPU) -> unconnected-(U7F-VDD_MPU-PadF13)
- U7 pad F4: Net-(U7F-VDDS_DDR) -> unconnected-(U7F-VDDS_DDR-PadF4)
- U7 pad F8: Net-(U7A-SYS_VDD3_3P3V@1) -> Net-(Q1-E)
- U7 pad F9: Net-(U7A-SYS_VDD3_3P3V@1) -> Net-(Q1-E)
- U7 pad G1: Net-(U7D-LCD_DATA2) -> Net-(J6-Pin_1)
- U7 pad G13: Net-(U7F-VDDS_PLL) -> unconnected-(U7F-VDDS_PLL-PadG13)
- U7 pad G2: Net-(U7D-LCD_DATA1) -> Net-(R25-22)
- U7 pad G3: Net-(U7D-LCD_DATA0) -> Net-(R25-11)
- U7 pad G4: Net-(U7F-VDD_CORE) -> unconnected-(U7F-VDD_CORE-PadG4)
- U7 pad G8: Net-(U7A-SYS_VDD3_3P3V@1) -> Net-(Q1-E)
- U7 pad G9: Net-(U7A-SYS_VDD3_3P3V@1) -> Net-(Q1-E)
- U7 pad H2: Net-(U7D-LCD_DATA4) -> Net-(R24-66)
- U7 pad H3: Net-(U7D-LCD_DATA3) -> Net-(R24-33)
- U7 pad H7: Net-(U7A-SYS_VDD3_3P3V@1) -> Net-(Q1-E)
- U7 pad H8: Net-(U7A-SYS_VDD3_3P3V@1) -> Net-(Q1-E)
- U7 pad H9: Net-(U7A-SYS_VDD3_3P3V@1) -> Net-(Q1-E)
- U7 pad J16: /SIP A, E ,F/VIN_USB -> Net-(U1-VCC)
- U7 pad J7: Net-(U7A-SYS_VDD3_3P3V@1) -> Net-(Q1-E)
- U7 pad J8: Net-(U7A-SYS_VDD3_3P3V@1) -> Net-(Q1-E)
- U7 pad J9: Net-(U7A-SYS_VDD3_3P3V@1) -> Net-(Q1-E)
- U7 pad K11: 3.3VA -> Net-(Q1-C)
- U7 pad K8: Net-(U7A-SYS_VDD3_3P3V@1) -> Net-(Q1-E)
- U7 pad K9: Net-(U7A-SYS_VDD3_3P3V@1) -> Net-(Q1-E)
- U7 pad L11: 3.3VA -> Net-(Q1-C)
- U7 pad L8: Net-(U7A-SYS_VDD3_3P3V@1) -> Net-(Q1-E)
- U7 pad L9: Net-(U7A-SYS_VDD3_3P3V@1) -> Net-(Q1-E)
- U7 pad M2: Net-(U7A-EEPROM_WP) -> /SIP A/EEPROM_WP
- U7 pad P9: /SIP A, E ,F/VIN_USB -> /V_USB
- U7 pad R11: Net-(U4-Y) -> /SIP A/nRESET
- U7 pad R9: /SIP A, E ,F/VIN_USB -> /V_USB
- U7 pad T9: /SIP A, E ,F/VIN_USB -> /V_USB
- Y1 pad 2: GND -> /SIP B/OSC0_GND
- Y1 pad 4: GND -> /SIP B/OSC0_GND
Routing:
- net Net-(J6-Pin_1): track 0.00 -> 151.0 mm, vias 0 -> 6
- net /Camera Logical Level Shifters/D3_I: track 0.00 -> 106.7 mm, vias 0 -> 4
- net Net-(U7D-LCD_DATA2): track 80.4 -> 0.00 mm, vias 3 -> 0
- net Net-(R24-88): track 70.6 -> 0.00 mm, vias 3 -> 0
- net Net-(Q1-C): track 0.00 -> 65.5 mm, vias 0 -> 4
- net /Camera Logical Level Shifters/D1_I: track 52.2 -> 110.5 mm, vias 1 -> 4
- net /Camera Logical Level Shifters/D0_I: track 48.3 -> 105.3 mm, vias 1 -> 4
- net Net-(J100-DAT2): track 56.6 -> 0.00 mm, vias 2 -> 0
- net 3.3VA: track 56.2 -> 0.00 mm, vias 3 -> 0
- net Net-(J100-DAT3/CS): track 55.2 -> 0.00 mm, vias 2 -> 0
- net /SIP C/D3_I: track 54.4 -> 0.00 mm, vias 1 -> 0
- net /Camera Logical Level Shifters/D2_I: track 50.1 -> 101.5 mm, vias 1 -> 4
- net Net-(J100-DAT0/DO): track 50.5 -> 0.00 mm, vias 2 -> 0
- net Net-(J100-DAT1): track 49.7 -> 0.00 mm, vias 2 -> 0
- net Net-(U7D-LCD_DATA0): track 42.4 -> 0.00 mm, vias 1 -> 0
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- added copper zone on F.Cu, net (none)
- added copper zone on F.Cu, net /V_USB
- added copper zone on In2.Cu, net /V_USB
- added copper zone on F.Cu, net Net-(Q1-E)
- removed copper zone on F.Cu, net /SIP A, E ,F/VIN_USB
- removed copper zone on In2.Cu, net /SIP A, E ,F/VIN_USB
- removed copper zone on F.Cu, net 3.3VA
- removed copper zone on F.Cu, net Net-(U7A-SYS_VDD3_3P3V@1)

Commit message: Routine push
Parts:
- removed TP183, TP184: TEST-POINT3X4, oresat-misc:TestPoint_Pad_D1.0mm
- added C48: 100n, oresat-passives:0603-C-NOSILK, F.Cu at (209.6, 94.6)
- added C49: 10n, oresat-passives:0603-C-NOSILK, F.Cu at (209.6, 96.7)
- added C71: 100n, oresat-passives:0603-C-NOSILK, F.Cu at (209.6, 98.8)
- moved C41 134.0 mm to (212.5, 80.1)
- moved C44 134.0 mm to (212.5, 82.2)
- moved C47 134.0 mm to (207.6, 67.7)
- moved C65 134.0 mm to (207.6, 69.8)
- moved C7 134.0 mm to (212.5, 78.0)
- moved C93 134.0 mm to (212.1, 68.8)
- moved R75 134.0 mm to (212.8, 84.6)
- moved R77 134.0 mm to (212.8, 87.1)
- moved R78 134.0 mm to (207.6, 71.9)
- moved TP109 134.0 mm to (207.4, 106.2)
- moved TP32 134.0 mm to (207.4, 110.5)
- moved J6 123.3 mm to (202.5, 73.3)
- moved J7 88.9 mm to (178.1, 79.8)
- moved R74 87.2 mm to (160.7, 90.2), turned to -90 degrees
- moved C29 3.63 mm to (148.9, 89.5)
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Connections:
- J4 pad 33: Net-(J4-Pad33) -> unconnected-(J4-Pad33)
- J4 pad 34: Net-(J4-Pad33) -> unconnected-(J4-Pad34)
- J4 pad 35: Net-(J4-Pad35) -> unconnected-(J4-Pad35)
- J4 pad 36: Net-(J4-Pad35) -> unconnected-(J4-Pad36)
Routing:
- net (no net): track 206.7 -> 2.54 mm, vias 1 -> 0
- net Net-(J6-Pin_1): track 151.0 -> 36.2 mm, vias 6 -> 2
- net /C3-UART-TX: track 179.6 -> 84.4 mm
- net GND: track 137.9 -> 44.8 mm, vias 278 -> 271
- net Net-(R25-11): track 107.6 -> 39.5 mm, vias 4 -> 3
- net unconnected-(U7B-USB1_VBUS-PadM15): track 58.1 -> 0.00 mm, vias 1 -> 0
- net unconnected-(U7B-USB1_DRVVBUS-PadM14): track 53.9 -> 0.00 mm, vias 1 -> 0
- net unconnected-(U7B-TDO-PadC2): track 46.8 -> 0.00 mm, vias 1 -> 0
- net unconnected-(U7B-TDI-PadC1): track 46.8 -> 0.00 mm, vias 1 -> 0
- net unconnected-(U7B-USB1_DM-PadL16): track 45.8 -> 0.00 mm, vias 2 -> 0
- net unconnected-(U7B-USB1_DP-PadL15): track 44.8 -> 0.00 mm, vias 2 -> 0
- net /SIP A/EEPROM_WP: track 29.5 -> 0.00 mm, vias 1 -> 0
- net unconnected-(R25-33-Pad3): track 13.1 -> 1.20 mm
- net Net-(R10-99): track 37.4 -> 25.9 mm
- net Net-(R25-22): track 46.6 -> 37.4 mm, vias 2 -> 3
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