File: hardware/star-tracker-card/star-tracker-card_5.kicad_sch (KiCad schematic)
At the start: 33 parts, among them Q1 MMBT2907, U10 TLVH431, U4 SN74LVC1G07DCK, U7 OSD3358-512M-BSM

Commit message: Star Tracker v1.3 files, including new Makefile, Readme, and fixes in ERC, DRC, and layout
Parts:
- Q1: DPN 5399-MMBT2907CT-ND -> 1727-2958-1-ND; MFR Shenzhen Slkormicro Semicon Co., Ltd. -> Nexperia; MPN MMBT2907 -> PMBT2907A,215
Changed lines of the file:
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@@
 	(title_block
 		(title "OreSat Star Tracker")
-		(date "2026-04-15")
+		(date "2026-04-22")
 		(rev "1.3")
 		(company "Portland State Aerospace Society")
@@
 			)
 		)
-		(property "Datasheet" "https://mm.digikey.com/Volume0/opasdata/d220001/medias/docus/6778/5399_MMBT2907%20SOT-23.PDF"
+		(property "Datasheet" "https://assets.nexperia.com/documents/data-sheet/PMBT2907A.pdf"
 			(at 213.36 130.81 0)
 			(hide yes)
@@
 			)
 		)
-		(property "Description" "Bipolar (BJT) Transistor PNP 40 V 600 mA 200MHz 250 mW Surface Mount SOT-23"
+		(property "Description" "Bipolar (BJT) Transistor PNP 60 V 600 mA 200MHz 250 mW Surface Mount TO-236AB"
 			(at 213.36 130.81 0)
 			(hide yes)
@@
 			)
 		)
-		(property "DPN" "5399-MMBT2907CT-ND"
+		(property "DPN" "1727-2958-1-ND"
 			(at 213.36 130.81 0)
 			(hide yes)
@@
 			)
 		)
-		(property "MFR" "Shenzhen Slkormicro Semicon Co., Ltd."
+		(property "MFR" "Nexperia"
 			(at 213.36 130.81 0)
 			(hide yes)
@@
 			)
 		)
-		(property "MPN" "MMBT2907"
+		(property "MPN" "PMBT2907A,215"
 			(at 213.36 130.81 0)
 			(hide yes)
