File: hardware/star-tracker-card/star-tracker-card_5.kicad_sch (KiCad schematic)
At the start: 33 parts, among them Q1 MMBT2907, U10 TLVH431, U4 SN74LVC1G07DCK, U7 OSD3358-512M-BSM

Commit message: Updates to BOM to get v1.3r1
All transistors upgraded, OPD circuit breaker cutoff raised to 924 mA.
Parts:
- Q1: value MMBT2907 -> PMBT2907,215; DPN 1727-2958-1-ND -> 1727-5176-1-ND; MPN PMBT2907A,215 -> PMBT2907,215
Other:
- note added: ""3.3V""
- note removed: "3.3V"
Changed lines of the file:
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@@
 		)
 	)
-	(text "3.3V"
+	(text "\"3.3V\""
 		(exclude_from_sim no)
-		(at 225.044 90.424 0)
+		(at 210.566 90.424 0)
 		(effects
 			(font
 				(size 1.27 1.27)
-				(thickness 0.254)
-				(bold yes)
+				(thickness 0.1588)
 			)
 		)
@@
 			)
 		)
-		(property "Value" "MMBT2907"
+		(property "Value" "PMBT2907,215"
 			(at 213.36 135.89 0)
 			(show_name no)
@@
 			)
 		)
-		(property "Datasheet" "https://assets.nexperia.com/documents/data-sheet/PMBT2907A.pdf"
+		(property "Datasheet" "https://assets.nexperia.com/documents/data-sheet/PMBT2907.pdf"
 			(at 213.36 130.81 0)
 			(hide yes)
@@
 			)
 		)
-		(property "Description" "Bipolar (BJT) Transistor PNP 60 V 600 mA 200MHz 250 mW Surface Mount TO-236AB"
+		(property "Description" "Bipolar (BJT) Transistor PNP 40 V 600 mA 200MHz 250 mW Surface Mount TO-236AB"
 			(at 213.36 130.81 0)
 			(hide yes)
@@
 			)
 		)
-		(property "DPN" "1727-2958-1-ND"
+		(property "DPN" "1727-5176-1-ND"
 			(at 213.36 130.81 0)
 			(hide yes)
@@
 			)
 		)
-		(property "MPN" "PMBT2907A,215"
+		(property "MPN" "PMBT2907,215"
 			(at 213.36 130.81 0)
 			(hide yes)
