File: hardware/star-tracker-2.0/star-tracker-2.0-card/star-tracker-card.kicad_sch (KiCad schematic)
At the start: 9 parts, among them J1 TFM-120-01-L-D-RA, J2 SM14B-SHLS-TF, J3 GRPB041VWVN-RC, J4 3-2492104-6

Commit message: Updated USB clamp
minor routing and schematic changes. Updated OPD with new transistors. Changed resistor values on LEDs.
Connections:
- net SIP A/nRESET: now also J2.10 (NRST)
- no-connect marks 25 -> 24
Other:
- sheet SIP A ports: added nRESET_CLAMP; removed none
- sheet SIP B ports: added nRESET_CLAMP; removed nRESET
Changed lines of the file:
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@@
 	)
 	(no_connect
-		(at 57.15 161.29)
-	)
-	(no_connect
 		(at 46.99 27.94)
 	)
@@
 	(wire
 		(pts
-			(xy 176.53 228.6) (xy 176.53 201.93)
-		)
-		(stroke
-			(width 0)
-			(type default)
-		)
-	)
-	(wire
-		(pts
 			(xy 48.26 55.88) (xy 190.5 55.88)
 		)
@@
 	(wire
 		(pts
+			(xy 134.62 222.25) (xy 95.25 222.25)
+		)
+		(stroke
+			(width 0)
+			(type default)
+		)
+	)
+	(wire
+		(pts
 			(xy 62.23 85.09) (xy 62.23 86.36)
 		)
@@
 	(wire
 		(pts
+			(xy 95.25 222.25) (xy 95.25 161.29)
+		)
+		(stroke
+			(width 0)
+			(type default)
+		)
+	)
+	(wire
+		(pts
 			(xy 234.95 144.78) (xy 265.43 144.78)
 		)
@@
 	(wire
 		(pts
+			(xy 176.53 224.79) (xy 176.53 201.93)
+		)
+		(stroke
+			(width 0)
+			(type default)
+		)
+	)
+	(wire
+		(pts
 			(xy 308.61 157.48) (xy 391.16 157.48)
 		)
@@
 	(wire
 		(pts
+			(xy 167.64 224.79) (xy 176.53 224.79)
+		)
+		(stroke
+			(width 0)
+			(type default)
+		)
+	)
+	(wire
+		(pts
 			(xy 46.99 91.44) (xy 49.53 91.44)
 		)
@@
 	(wire
 		(pts
-			(xy 49.53 83.82) (xy 49.53 86.36)
+			(xy 57.15 161.29) (xy 95.25 161.29)
 		)
 		(stroke
 			(width 0)
-			(type solid)
+			(type default)
 		)
 	)
 	(wire
 		(pts
-			(xy 87.63 229.87) (xy 134.62 229.87)
+			(xy 49.53 83.82) (xy 49.53 86.36)
 		)
 		(stroke
 			(width 0)
-			(type default)
+			(type solid)
 		)
 	)
 	(wire
 		(pts
-			(xy 167.64 228.6) (xy 176.53 228.6)
+			(xy 87.63 229.87) (xy 134.62 229.87)
 		)
 		(stroke
@@
 			)
 		)
-		(pin "nRESET" input
+		(pin "nRESET_CLAMP" input
 			(at 167.64 201.93 0)
 			(effects
@@
 		)
 		(pin "nRESET" output
-			(at 167.64 228.6 0)
+			(at 134.62 222.25 180)
+			(effects
+				(font
+					(size 1.27 1.27)
+				)
+				(justify left)
+			)
+		)
+		(pin "nRESET_CLAMP" output
+			(at 167.64 224.79 0)
 			(effects
 				(font
