File: hardware/star-tracker-2.0/star-tracker-2.0-card/star-tracker-card_5.kicad_sch (KiCad schematic)
At the start: 21 parts, among them Q6 MMBT2907, U7 OSD3358-512M-BSM, U8 SN74LVC1G07DCK, U9 TLVH431

Commit message: Updated USB clamp
minor routing and schematic changes. Updated OPD with new transistors. Changed resistor values on LEDs.
Parts:
- R46: value 1k -> 10k; DPN RMCF0603FT2K70CT-ND -> RMCF0603FT10K0CT-ND; MPN RMCF0603FT1K00 -> RMCF0603FT10K0
Changed lines of the file:
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@@
+	)
+	(junction
+		(at 300.99 217.17)
+		(diameter 0)
+		(color 0 0 0 0)
 	)
 	(junction
@@
 	(wire
 		(pts
+			(xy 300.99 217.17) (xy 300.99 222.25)
+		)
+		(stroke
+			(width 0)
+			(type default)
+		)
+	)
+	(wire
+		(pts
 			(xy 248.92 189.23) (xy 248.92 186.69)
 		)
@@
 	(wire
 		(pts
+			(xy 300.99 217.17) (xy 303.53 217.17)
+		)
+		(stroke
+			(width 0)
+			(type default)
+		)
+	)
+	(wire
+		(pts
 			(xy 289.56 151.13) (xy 274.32 151.13)
 		)
@@
 	(wire
 		(pts
-			(xy 287.02 217.17) (xy 290.83 217.17)
+			(xy 287.02 217.17) (xy 300.99 217.17)
 		)
 		(stroke
@@
 			)
 			(justify left bottom)
+		)
+	)
+	(hierarchical_label "nRESET_CLAMP"
+		(shape output)
+		(at 300.99 222.25 270)
+		(effects
+			(font
+				(size 1.27 1.27)
+			)
+			(justify right)
 		)
 	)
@@
 	(hierarchical_label "nRESET"
 		(shape output)
-		(at 290.83 217.17 0)
+		(at 303.53 217.17 0)
 		(effects
 			(font
@@
 			)
 		)
-		(property "Value" "1k"
+		(property "Value" "10k"
 			(at 283.464 85.852 0)
 			(show_name no)
@@
 					(size 1.27 1.27)
 				)
-				(justify right bottom)
+				(justify right top)
 			)
 		)
@@
 			)
 		)
-		(property "Description" "1 kOhms ±1% 0.1W, 1/10W Chip Resistor 0603 (1608 Metric) Automotive AEC-Q200 Thick Film"
+		(property "Description" "10 kOhms ±1% 0.1W, 1/10W Chip Resistor 0603 (1608 Metric) Automotive AEC-Q200 Thick Film"
 			(at 279.4 83.82 0)
 			(hide yes)
@@
 			)
 		)
-		(property "DPN" "RMCF0603FT2K70CT-ND"
+		(property "DPN" "RMCF0603FT10K0CT-ND"
 			(at 279.4 83.82 0)
 			(hide yes)
@@
 			)
 		)
-		(property "MPN" "RMCF0603FT1K00"
+		(property "MPN" "RMCF0603FT10K0"
 			(at 279.4 83.82 0)
 			(hide yes)
