File: hardware/star-tracker-2.0/star-tracker-2.0-card/star-tracker-card_3.kicad_sch (KiCad schematic)
At the start: 40 parts, among them J5 DM3BT-DSF-PEJS, U11 ICM-42688-P, U12 TCAN330, U13 EMMC+RESET+5.1-COMPATIBLE-BA, U7 OSD3358-512M-BSM

Commit message: Replaced IMU with BMI component from bosch
ported over changes from schematic to pcb. Removed old connectors page.
Parts:
- removed C30: 10n, oresat-passives:0603-C-NOSILK, symbol Device:C_Small
- removed C31: 2.2u, oresat-passives:0603-C-NOSILK, symbol Device:C_Small
- removed U11: ICM-42688-P, oresat-ics:PQFN50P300X250X97-14N, symbol oresat-ics:ICM-42688-P
- added C53: 100n, oresat-passives:0603-C-NOSILK, symbol Device:C_Small
- added U11: BMI270, oresat-ics:PQFN50P300X250X97-14N, symbol oresat-ics:BMI270
Connections:
- net 3.3V: now also C53.1, U11.5 (VDD_IO), U11.8 (VDD)
- net GND: now also C53.2, U11.10 (OCSB), U11.11 (OSDO), U11.6 (GND_IO), U11.7 (GND)
- net IMU_I2C1_SCLK: now also U11.13 (SCX)
- net IMU_I2C1_SDA: now also U11.14 (SDX)
- net IMU_INT1: now also U11.4 (INT1)
- net IMU_INT2: now also U11.9 (INT2)
- net at R59.1: now also U11.12 (CSB)
- net at R58.2: now also U11.1 (SDO)
